File: ESP32.kicad_sch (KiCad schematic)
At the start: 15 parts, among them J5 USB_B, Q2 MMBT3904, Q3 MMBT3904, U1 CH340C, U3 MCP1700x-330xxMB, U4 ESP32-S3-WROOM-2

Commit message: update
Parts:
- added D3: D, symbol Device:D
Connections:
- net +5V: now also D3.2 (A); no longer C2.1, U3.2 (VI)
- net 10m band en: no longer names the net of U4.22 (IO14)
- net 12m band en: no longer names the net of U4.21 (IO13)
- net 15m band en: no longer names the net of U4.20 (IO12)
- net 17m band en: no longer names the net of U4.19 (IO11)
- net 20m band en renamed Iambic Paddle Dah
- net 30m band en renamed Iambic Paddle Dit
- net 40m band en renamed Filter 2 En
- net 80m band en renamed Filter 1 En
- new net Vdrive: C2.1, D3.1 (K), U3.2 (VI)
- no-connect marks 25 -> 29
