File: RP2040.kicad_sch (KiCad schematic)
At the start: 30 parts, among them J6 USB_C_Receptacle_USB2.0_14P, U1 MCP1700x-330xxMB, U2 W25Q128JVS, U3 RP2040, Y1 ABM8-272-T3

Commit message: some big updates
Parts:
- added R2, R3: 5k1, Resistor_SMD:R_0603_1608Metric, symbol Device:R
- C1, C2: footprint Capacitor_SMD:C_1206_3216Metric -> Capacitor_SMD:C_0603_1608Metric
- C10, C11, C12, C13, C14, C15, C16, C3, C4, C5, C6, C7, C8, C9: footprint (none) -> Capacitor_SMD:C_0603_1608Metric
- D2: footprint Diode_SMD:D_1206_3216Metric -> (none)
- JP1: footprint Jumper:SolderJumper-2_P1.3mm_Open_RoundedPad1.0x1.5mm -> (none)
- R10: renamed from R8; footprint Resistor_SMD:R_1206_3216Metric -> Resistor_SMD:R_0603_1608Metric
- R4: renamed from R2; footprint (none) -> Resistor_SMD:R_0603_1608Metric
- R5: renamed from R3; footprint (none) -> Resistor_SMD:R_0603_1608Metric
- R6: renamed from R4; footprint (none) -> Resistor_SMD:R_0603_1608Metric
- R7: renamed from R5; footprint (none) -> Resistor_SMD:R_0603_1608Metric
- R8: renamed from R6; footprint (none) -> Resistor_SMD:R_0603_1608Metric
- R9: renamed from R7; footprint Resistor_SMD:R_1206_3216Metric -> Resistor_SMD:R_0603_1608Metric
- U1: footprint Package_TO_SOT_SMD:SOT-89-3 -> (none)
- U2: footprint Package_SO:SOIC-8_5.23x5.23mm_P1.27mm -> (none)
- U3: footprint Package_DFN_QFN:QFN-56-1EP_7x7mm_P0.4mm_EP3.2x3.2mm -> (none)
Connections:
- net +3V3 is gone; now on net +3.3V: C10.1, C11.1, C12.1, C13.1, C14.1, C15.1, C16.1, C3.1, C9.1, R5.1, U2.8 (VCC), U3.1 (IOVDD), U3.10 (IOVDD), U3.22 (IOVDD), U3.33 (IOVDD), U3.42 (IOVDD), U3.43 (ADC_AVDD), U3.44 (VREG_IN), U3.48 (USB_VDD), U3.49 (IOVDD)
- net GND: now also R2.2, R3.2
- net at J6.A5 (CC1): now also R3.1
- net at J6.B5 (CC2): now also R2.1
- no-connect marks 23 -> 27
