File: CW HF Transceiver.kicad_sch (KiCad schematic)
At the start: 6 parts, among them J2 ANT out, J3 Vin, J4 Automated pulses, Q1 S8550, SW1 SW_Push

Commit message: a
Connections:
- net Filtering/wave: now also Q1.3 (C)
- net tx: now reaches J2.1 (In)
- net tx: no longer Q1.3 (C)
- net filtered renamed Square Wave Gen/wave out
Other:
- note added: "Note: Morse input is held low, but can be pulled high by the header for a morse key, the esp32 or the built-in button."
- moved on the sheet: Q1

Commit message: update
Parts:
- removed Q1: S8550, Package_TO_SOT_THT:TO-39-3_Window, symbol Transistor_BJT:S8550
- removed SW1: SW_Push, Button_Switch_SMD:SW_Push_1P1T_NO_6x6mm_H9.5mm, symbol Switch:SW_Push
- added D2: D_Zener, symbol Device:D_Zener
- added J1: AudioJack2, symbol Connector_Audio:AudioJack2
- added J6: AudioJack3, symbol Connector_Audio:AudioJack3
- added Q1: DMN13H750S, Package_TO_SOT_SMD:SOT-23, symbol Transistor_FET:DMN13H750S
- J2: value ANT out -> BNC
- J4: value Automated pulses -> Morse Key
- R1: value 4.7k -> R; footprint Resistor_SMD:R_1206_3216Metric -> (none)
Connections:
- net Mouse Input is gone; now on net VCC: R1.1
- net GND: now also J4.1 (Pin_1), D2.2 (A), J1.S, J6.S; no longer R1.2
- net Morse Input: now also J4.2 (Pin_2), J1.T, Q1.1 (G); no longer J4.1 (Pin_1)
- net VCC: no longer J4.2 (Pin_2)
- new net Amplifier/Rx: Q1.3 (D)
- new net Vdrive: D2.1 (K), R1.2
- new net dah: J6.T
- new net dit: J6.R
Other:
- added sheet Amplifier (Amplifier.kicad_sch)
- sheet ESP32 Driver: file untitled.kicad_sch -> ESP32.kicad_sch
- sheet ESP32 Driver ports: added Filter 1 En, Filter 2 En, Iambic Paddle Dah, Iambic Paddle Dit; removed 10m band en, 12m band en, 15m band en, 17m band en, 20m band en, 30m band en, 40m band en, 80m band en
- sheet Filtering ports: added Filter 1 En, Filter 2 En; removed 10m band en, 12m band en, 15m band en, 17m band en, 20m band en, 30m band en, 40m band en, 80m band en
- note added: "Note: Iambic paddle: 3 Pin audio connector Morse key: 2 Pin audio connector"
- note removed: "Note: Morse input is held low, but can be pulled high by the header for a morse key, the esp32 or the built-in button."

Commit message: update amplifier
Connections:
- net Amplifier/Rx: now also Q1.2 (S); no longer Q1.3 (D)
Other:
- moved on the sheet: Q1
Changed lines of the file:
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@@
 	(symbol
 		(lib_id "Transistor_FET:DMN13H750S")
-		(at 150.114 78.74 180)
+		(at 150.114 78.74 0)
+		(mirror y)
 		(unit 1)
 		(exclude_from_sim no)
@@
 		(on_board yes)
 		(dnp no)
-		(fields_autoplaced yes)
 		(property "Reference" "Q1"
-			(at 143.764 77.4699 0)
+			(at 143.764 80.0101 0)
 			(effects
 				(font
@@
 		)
 		(property "Value" "DMN13H750S"
-			(at 143.764 80.0099 0)
+			(at 143.764 77.4701 0)
 			(effects
 				(font
@@
 		)
 		(property "Footprint" "Package_TO_SOT_SMD:SOT-23"
-			(at 145.034 76.835 0)
+			(at 145.034 80.645 0)
 			(effects
 				(font
@@
 		)
 		(property "Datasheet" "http://www.diodes.com/assets/Datasheets/DMN13H750S.pdf"
-			(at 145.034 74.93 0)
+			(at 145.034 82.55 0)
 			(effects
 				(font

Commit message: some big updates
Parts:
- removed J2: BNC, Connector_Coaxial:BNC_Amphenol_B6252HB-NPP3G-50_Horizontal, symbol Connector:Conn_Coaxial
- removed J3: Vin, TerminalBlock:TerminalBlock_Altech_AK300-2_P5.00mm, symbol Connector:Screw_Terminal_01x02
- removed J4: Morse Key, TerminalBlock:TerminalBlock_Altech_AK300-2_P5.00mm, symbol Connector:Screw_Terminal_01x02
- removed Q1: DMN13H750S, Package_TO_SOT_SMD:SOT-23, symbol Transistor_FET:DMN13H750S
- added J1: Barrel_Jack, symbol Connector:Barrel_Jack
- added J5: Conn_Coaxial, symbol Connector:Conn_Coaxial
- added R12: 4.7k, Resistor_SMD:R_0603_1608Metric, symbol Device:R
- R1: footprint (none) -> Resistor_SMD:R_0603_1608Metric
- renumbered D2 to D1, J1 to J3, J6 to J4
Connections:
- net GND: now also J1.2, J5.2 (Ext)
- net Morse Input: now also R12.2
- net VCC: now also J1.1
- net tx: now also J5.1 (In)
- new net +3.3V: R12.1
- no-connect marks 0 -> 1
Other:
- sheet ESP32 Driver renamed RP2040 Driver
- added sheet IO (IO.kicad_sch)
- added sheet Receiver (Receiver.kicad_sch)
- sheet Amplifier ports: added 0º Wave, 180º Wave, Amp enable, Amplified; removed Rx, Tx
- sheet RP2040 Driver: file ESP32.kicad_sch -> RP2040.kicad_sch
- sheet Square Wave Gen ports: added 180º Wave Out, BFO out, Wave out; removed wave out
- note removed: "Note: Iambic paddle: 3 Pin audio connector Morse key: 2 Pin audio connector"
- title: (none) -> CW HF Transceiver
- moved on the sheet: D1, R1

Commit message: update
Parts:
- removed J3: AudioJack2, symbol Connector_Audio:AudioJack2
- added R2: 4.7k, Resistor_SMD:R_0603_1608Metric, symbol Device:R
- R1: value R -> 4.7k
- renumbered J4 to J2, J5 to J3, R12 to R3
Connections:
- net +3.3V: now also R1.1, R2.1
- net VCC: now also D1.1 (K); no longer R1.1
- net dah: now also R2.2
- net dit: now also R1.2
- removed net Vdrive: D1.1 (K), R1.2
Other:
- sheet RP2040 Driver renamed STM32 Driver
- sheet STM32 Driver: file RP2040.kicad_sch -> STM32 Driver.kicad_sch
- moved on the sheet: J2
