File: IO.kicad_sch (KiCad schematic)
At the start: 2 parts, among them SW1 VFO

Commit message: update
Other:
- note added: "TODO: plan & make IO"
Changed lines of the file:
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@@
+		)
+	)
+	(text "TODO: plan & make IO"
+		(exclude_from_sim no)
+		(at 109.474 66.548 0)
+		(effects
+			(font
+				(size 1.27 1.27)
+			)
 		)
 	)
@@
 		(dnp no)
 		(fields_autoplaced yes)
-		(property "Reference" "#PWR050"
+		(property "Reference" "#PWR041"
 			(at 97.79 87.63 0)
 			(effects
@@
 			(project ""
 				(path "/46807950-96a2-445b-a4f1-43cb63a530a8/619a8caf-8757-451b-80db-58c150aafaca"
-					(reference "#PWR050")
+					(reference "#PWR041")
 					(unit 1)
 				)
