File: STM32 Driver.kicad_sch (KiCad schematic)
At the start: 18 parts, among them J4 USB_C_Receptacle_USB2.0_14P, U1 MCP1700x-330xxMB, U2 STM32F072C8Tx, U7 USB6B1

Commit message: on the final bits!
Parts:
- removed TP1: SWDIO, symbol Connector:TestPoint
- removed TP8: SWCLK, symbol Connector:TestPoint
- added J5: JTAG, symbol Connector:Conn_01x04_Pin
- renumbered D2 to D1, U7 to U1, U1 to U2, U2 to U3
Connections:
- net +3.3V: now also J5.4 (Pin_4)
- net Filter 1 En: now also U3.19 (PB1); no longer U3.42 (PB6)
- net Filter 2 En: now also U3.20 (PB2); no longer U3.43 (PB7)
- net GND: now also J5.3 (Pin_3)
- net encoded out: now also U3.18 (PB0); no longer U3.41 (PB5)
- net at U3.34 (PA13): now also J5.2 (Pin_2)
- net at U3.37 (PA14): now also J5.1 (Pin_1)
- net Filter 3 En: now reaches U3.39 (PB3)
- no-connect marks 28 -> 23

Commit message: should be done
Parts:
- added J6: Conn_02x12_Counter_Clockwise, symbol Connector_Generic:Conn_02x12_Counter_Clockwise
- renumbered C1 to C2, C2 to C3, C3 to C4, C4 to C5, C5 to C6, C6 to C7, C7 to C8, D1 to D2, R4 to R3, R5 to R4, R6 to R5, R7 to R6
Connections:
- net encoded out is gone; now on net Filter 1 En: U3.18 (PB0)
- net +3.3V: now also J6.24 (Pin_24)
- net Filter 1 En: no longer U3.19 (PB1)
- net Filter 2 En: now also U3.19 (PB1); no longer U3.20 (PB2)
- net Filter 3 En: now also U3.20 (PB2); no longer U3.39 (PB3)
- net GND: now also J6.1 (Pin_1), J6.2 (Pin_2)
- net scl: now also J6.7 (Pin_7)
- net sda: now also J6.8 (Pin_8)
- net PA2: now reaches U3.12 (PA2)
- net PA2: now also J6.21 (Pin_21)
- net PA3: now reaches U3.13 (PA3)
- net PA3: now also J6.20 (Pin_20)
- net PA4: now reaches U3.14 (PA4)
- net PA4: now also J6.19 (Pin_19)
- net PA5: now reaches U3.15 (PA5)
- net PA5: now also J6.18 (Pin_18)
- net PA6: now reaches U3.16 (PA6)
- net PA6: now also J6.17 (Pin_17)
- net PA7: now reaches U3.17 (PA7)
- net PA7: now also J6.16 (Pin_16)
- net PB10: now reaches U3.21 (PB10)
- net PB10: now also J6.9 (Pin_9)
- net PB11: now reaches U3.22 (PB11)
- net PB11: now also J6.10 (Pin_10)
- net PB12: now reaches U3.25 (PB12)
- net PB12: now also J6.11 (Pin_11)
- net PB13: now reaches U3.26 (PB13)
- net PB13: now also J6.12 (Pin_12)
- net PB14: now reaches U3.27 (PB14)
- net PB14: now also J6.23 (Pin_23)
- net PB15: now reaches U3.28 (PB15)
- net PB15: now also J6.22 (Pin_22)
- net PA8: now reaches U3.29 (PA8)
- net PA8: now also J6.15 (Pin_15)
- net PA9: now reaches U3.30 (PA9)
- net PA9: now also J6.14 (Pin_14)
- net PA10: now reaches U3.31 (PA10)
- net PA10: now also J6.13 (Pin_13)
- net PB4: now reaches U3.40 (PB4)
- net PB4: now also J6.3 (Pin_3)
- net PB5: now reaches U3.41 (PB5)
- net PB5: now also J6.4 (Pin_4)
- net PB6: now reaches U3.42 (PB6)
- net PB6: now also J6.5 (Pin_5)
- net PB7: now reaches U3.43 (PB7)
- net PB7: now also J6.6 (Pin_6)
- new net Amp Enable: U3.39 (PB3)
- no-connect marks 23 -> 8
Other:
- note removed: "NOTE: switch will choose between iambic paddle & bug"

Commit message: add the pcb
Parts:
- removed C8: 100n, symbol Device:C
- removed D2: D, symbol Device:D
- removed J4: USB_C_Receptacle_USB2.0_14P, symbol Connector:USB_C_Receptacle_USB2.0_14P
- removed J6: Conn_02x12_Counter_Clockwise, symbol Connector_Generic:Conn_02x12_Counter_Clockwise
- added C9: 100n, Capacitor_SMD:C_0603_1608Metric, symbol Device:C
- added J2: Conn_02x12_Odd_Even, Connector_PinHeader_1.27mm:PinHeader_2x12_P1.27mm_Vertical_SMD, symbol Connector_Generic:Conn_02x12_Odd_Even
- added USBC1: USB3.1C16PFSMT, plib:USB-C-SMD_TYPE-C-USB-17, symbol plib:USB3.1C16PFSMT
- C5: renamed from C4; footprint (none) -> Capacitor_SMD:C_0603_1608Metric
- C6: renamed from C5; footprint (none) -> Capacitor_SMD:C_0603_1608Metric
- C7: renamed from C6; footprint (none) -> Capacitor_SMD:C_0603_1608Metric
- C8: renamed from C7; footprint (none) -> Capacitor_SMD:C_0603_1608Metric
- J1: renamed from J5; footprint (none) -> Connector_PinHeader_1.27mm:PinHeader_1x04_P1.27mm_Vertical
- U2: footprint (none) -> Package_TO_SOT_SMD:SOT-89-3
- renumbered C2 to C3, C3 to C4
Connections:
- net PB4 is gone; now on net Filter 1 En: U3.40 (PB4)
- net PB5 is gone; now on net Filter 2 En: U3.41 (PB5)
- net PB6 is gone; now on net Filter 3 En: U3.42 (PB6)
- net VBUS is gone; now on net +5V: U1.1 (VBUS), U1.8 (VBUS)
- net +3.3V: now also C9.1, J2.2 (Pin_2)
- net +5V: now also USBC1.A4 (VBUS), USBC1.A9 (VBUS)
- net D+: now also U1.7 (I/O1); no longer U1.6 (I/O2)
- net D-: now also U1.6 (I/O2); no longer U1.7 (I/O1)
- net Filter 1 En: no longer U3.18 (PB0)
- net Filter 2 En: no longer U3.19 (PB1)
- net Filter 3 En: no longer U3.20 (PB2)
- net GND: now also C9.2, J2.1 (Pin_1), J2.3 (Pin_3), USBC1.0, USBC1.A1 (GND), USBC1.A12 (GND)
- net PA10: now also J2.23 (Pin_23)
- net PA2: now also J2.5 (Pin_5)
- net PA3: now also J2.4 (Pin_4)
- net PA4: now also J2.6 (Pin_6)
- net PA5: now also J2.8 (Pin_8)
- net PA6: now also J2.10 (Pin_10)
- net PA7: now also J2.12 (Pin_12)
- net PA8: now also J2.19 (Pin_19)
- net PA9: now also J2.21 (Pin_21)
- net PB10: now also J2.14 (Pin_14)
- net PB11: now also J2.16 (Pin_16)
- net PB12: now also J2.18 (Pin_18)
- net PB13: now also J2.20 (Pin_20)
- net PB14: now also J2.22 (Pin_22)
- net PB15: now also J2.24 (Pin_24)
- net PB7: now also J2.11 (Pin_11)
- net scl: now also J2.9 (Pin_9)
- net sda: now also J2.7 (Pin_7)
- net at R4.1: now also USBC1.A5 (CC1)
- net at U1.3 (I/O2): now also USBC1.A7 (DN1), USBC1.B7 (DN2)
- net at U1.2 (I/O1): now also USBC1.A6 (DP1), USBC1.B6 (DP2)
- net at R3.1: now also USBC1.B5 (CC2)
- new net PB0: J2.13 (Pin_13), U3.18 (PB0)
- new net PB1: J2.15 (Pin_15), U3.19 (PB1)
- new net PB2: J2.17 (Pin_17), U3.20 (PB2)
- no-connect marks 8 -> 10
