File: Receiver.kicad_sch (KiCad schematic)
At the start: 11 parts, among them J7 AudioJack3, SW2 Reset RX, U7 Si4735-D60-GU, Y3 37.628KHz

Commit message: update
Parts:
- removed LS1: Speaker, symbol Device:Speaker
- renumbered C24 to C17, C25 to C18, C26 to C19, C27 to C20, C28 to C21, J7 to J5, R11 to R8, U7 to U6, Y3 to Y2
Other:
- moved on the sheet: J5
Changed lines of the file:
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@@
-	(wire
-		(pts
-			(xy 80.01 58.42) (xy 80.01 60.96)
-		)
-		(stroke
-			(width 0)
-			(type default)
-		)
-	)
 	(wire
 		(pts
@@
 	(wire
 		(pts
-			(xy 135.89 107.95) (xy 142.24 107.95)
+			(xy 135.89 107.95) (xy 140.97 107.95)
 		)
 		(stroke
@@
 	(wire
 		(pts
-			(xy 135.89 105.41) (xy 142.24 105.41)
+			(xy 135.89 105.41) (xy 140.97 105.41)
 		)
 		(stroke
@@
 	(wire
 		(pts
-			(xy 142.24 102.87) (xy 134.62 102.87)
+			(xy 140.97 102.87) (xy 134.62 102.87)
 		)
 		(stroke
@@
 		(dnp no)
 		(fields_autoplaced yes)
-		(property "Reference" "R11"
+		(property "Reference" "R8"
 			(at 59.69 63.4999 0)
 			(effects
@@
 			(project ""
 				(path "/46807950-96a2-445b-a4f1-43cb63a530a8/3d57e32e-3e27-4526-9430-25edad46b736"
-					(reference "R11")
+					(reference "R8")
 					(unit 1)
 				)
@@
 		(dnp no)
 		(fields_autoplaced yes)
-		(property "Reference" "#PWR056"
+		(property "Reference" "#PWR047"
 			(at 77.47 143.51 0)
 			(effects
@@
 			(project ""
 				(path "/46807950-96a2-445b-a4f1-43cb63a530a8/3d57e32e-3e27-4526-9430-25edad46b736"
-					(reference "#PWR056")
+					(reference "#PWR047")
 					(unit 1)
 				)
@@
 		(dnp no)
 		(fields_autoplaced yes)
-		(property "Reference" "#PWR058"
+		(property "Reference" "#PWR048"
 			(at 95.25 110.49 0)
 			(effects
@@
 			(project ""
 				(path "/46807950-96a2-445b-a4f1-43cb63a530a8/3d57e32e-3e27-4526-9430-25edad46b736"
-					(reference "#PWR058")
+					(reference "#PWR048")
 					(unit 1)
 				)
@@
 		(dnp no)
 		(fields_autoplaced yes)
-		(property "Reference" "#PWR052"
+		(property "Reference" "#PWR043"
 			(at 57.15 64.77 0)
 			(effects
@@
 			(project ""
 				(path "/46807950-96a2-445b-a4f1-43cb63a530a8/3d57e32e-3e27-4526-9430-25edad46b736"
-					(reference "#PWR052")
+					(reference "#PWR043")
 					(unit 1)
 				)
@@
 		(dnp no)
 		(fields_autoplaced yes)
-		(property "Reference" "C28"
+		(property "Reference" "C21"
 			(at 134.62 63.4999 0)
 			(effects
@@
 			(project "CW HF Transceiver"
 				(path "/46807950-96a2-445b-a4f1-43cb63a530a8/3d57e32e-3e27-4526-9430-25edad46b736"
-					(reference "C28")
-					(unit 1)
-				)
-			)
-		)
-	)
-	(symbol
-		(lib_id "Device:Speaker")
-		(at 147.32 87.63 0)
-		(unit 1)
-		(exclude_from_sim no)
-		(in_bom yes)
-		(on_board yes)
-		(dnp no)
-		(fields_autoplaced yes)
-		(property "Reference" "LS1"
-			(at 152.4 87.6299 0)
-			(effects
-				(font
-					(size 1.27 1.27)
-				)
-				(justify left)
-			)
-		)
-		(property "Value" "Speaker"
-			(at 152.4 90.1699 0)
-			(effects
-				(font
-					(size 1.27 1.27)
-				)
-				(justify left)
-			)
-		)
-		(property "Footprint" ""
-			(at 147.32 92.71 0)
-			(effects
-				(font
-					(size 1.27 1.27)
-				)
-				(hide yes)
-			)
-		)
-		(property "Datasheet" "~"
-			(at 147.066 88.9 0)
-			(effects
-				(font
-					(size 1.27 1.27)
-				)
-				(hide yes)
-			)
-		)
-		(property "Description" "Speaker"
-			(at 147.32 87.63 0)
-			(effects
-				(font
-					(size 1.27 1.27)
-				)
-				(hide yes)
-			)
-		)
-		(pin "2"
-		)
-		(pin "1"
-		)
-		(instances
-			(project ""
-				(path "/46807950-96a2-445b-a4f1-43cb63a530a8/3d57e32e-3e27-4526-9430-25edad46b736"
-					(reference "LS1")
+					(reference "C21")
 					(unit 1)
 				)
@@
 		(dnp no)
 		(fields_autoplaced yes)
-		(property "Reference" "#PWR053"
+		(property "Reference" "#PWR044"
 			(at 60.96 104.14 0)
 			(effects
@@
 			(project ""
 				(path "/46807950-96a2-445b-a4f1-43cb63a530a8/3d57e32e-3e27-4526-9430-25edad46b736"
-					(reference "#PWR053")
+					(reference "#PWR044")
 					(unit 1)
 				)
@@
 		(dnp no)
 		(fields_autoplaced yes)
-		(property "Reference" "C24"
+		(property "Reference" "C17"
 			(at 72.39 126.9999 0)
 			(effects
@@
 			(project ""
 				(path "/46807950-96a2-445b-a4f1-43cb63a530a8/3d57e32e-3e27-4526-9430-25edad46b736"
-					(reference "C24")
+					(reference "C17")
 					(unit 1)
 				)
@@
 		(dnp no)
 		(fields_autoplaced yes)
-		(property "Reference" "C26"
+		(property "Reference" "C19"
 			(at 105.41 63.4999 0)
 			(effects
@@
 			(project ""
 				(path "/46807950-96a2-445b-a4f1-43cb63a530a8/3d57e32e-3e27-4526-9430-25edad46b736"
-					(reference "C26")
+					(reference "C19")
 					(unit 1)
 				)
@@
 		(dnp no)
 		(fields_autoplaced yes)
-		(property "Reference" "#PWR055"
+		(property "Reference" "#PWR046"
 			(at 77.47 113.03 0)
 			(effects
@@
 			(project "CW HF Transceiver"
 				(path "/46807950-96a2-445b-a4f1-43cb63a530a8/3d57e32e-3e27-4526-9430-25edad46b736"
-					(reference "#PWR055")
+					(reference "#PWR046")
 					(unit 1)
 				)
@@
 		(dnp no)
 		(fields_autoplaced yes)
-		(property "Reference" "C25"
+		(property "Reference" "C18"
 			(at 90.17 126.9999 0)
 			(effects
@@
 			(project "CW HF Transceiver"
 				(path "/46807950-96a2-445b-a4f1-43cb63a530a8/3d57e32e-3e27-4526-9430-25edad46b736"
-					(reference "C25")
+					(reference "C18")
 					(unit 1)
 				)
@@
 	(symbol
 		(lib_id "Connector_Audio:AudioJack3")
-		(at 147.32 105.41 0)
+		(at 146.05 105.41 0)
 		(mirror y)
 		(unit 1)
@@
 		(on_board yes)
 		(dnp no)
-		(property "Reference" "J7"
-			(at 149.225 96.52 0)
+		(property "Reference" "J5"
+			(at 147.955 96.52 0)
 			(effects
 				(font
@@
 		)
 		(property "Value" "AudioJack3"
-			(at 149.225 99.06 0)
+			(at 147.955 99.06 0)
 			(effects
 				(font
@@
 		)
 		(property "Footprint" ""
-			(at 147.32 105.41 0)
+			(at 146.05 105.41 0)
 			(effects
 				(font
@@
 		)
 		(property "Datasheet" "~"
-			(at 147.32 105.41 0)
+			(at 146.05 105.41 0)
 			(effects
 				(font
@@
 		)
 		(property "Description" "Audio Jack, 3 Poles (Stereo / TRS)"
-			(at 147.32 105.41 0)
+			(at 146.05 105.41 0)
 			(effects
 				(font
@@
 			(project ""
 				(path "/46807950-96a2-445b-a4f1-43cb63a530a8/3d57e32e-3e27-4526-9430-25edad46b736"
-					(reference "J7")
+					(reference "J5")
 					(unit 1)
 				)
@@
 		(dnp no)
 		(fields_autoplaced yes)
-		(property "Reference" "#PWR054"
+		(property "Reference" "#PWR045"
 			(at 74.93 62.23 0)
 			(effects
@@
 			(project ""
 				(path "/46807950-96a2-445b-a4f1-43cb63a530a8/3d57e32e-3e27-4526-9430-25edad46b736"
-					(reference "#PWR054")
+					(reference "#PWR045")
 					(unit 1)
 				)
@@
 		(on_board yes)
 		(dnp no)
-		(property "Reference" "U7"
+		(property "Reference" "U6"
 			(at 82.2041 57.15 0)
 			(effects
@@
 			(project ""
 				(path "/46807950-96a2-445b-a4f1-43cb63a530a8/3d57e32e-3e27-4526-9430-25edad46b736"
-					(reference "U7")
-					(unit 1)
-				)
-			)
-		)
-	)
-	(symbol
-		(lib_id "power:+3.3V")
-		(at 80.01 58.42 0)
-		(unit 1)
-		(exclude_from_sim no)
-		(in_bom yes)
-		(on_board yes)
-		(dnp no)
-		(fields_autoplaced yes)
-		(property "Reference" "#PWR057"
-			(at 80.01 62.23 0)
-			(effects
-				(font
-					(size 1.27 1.27)
-				)
-				(hide yes)
-			)
-		)
-		(property "Value" "+3.3V"
-			(at 80.01 53.34 0)
-			(effects
-				(font
-					(size 1.27 1.27)
-				)
-			)
-		)
-		(property "Footprint" ""
-			(at 80.01 58.42 0)
-			(effects
-				(font
-					(size 1.27 1.27)
-				)
-				(hide yes)
-			)
-		)
-		(property "Datasheet" ""
-			(at 80.01 58.42 0)
-			(effects
-				(font
-					(size 1.27 1.27)
-				)
-				(hide yes)
-			)
-		)
-		(property "Description" "Power symbol creates a global label with name \"+3.3V\""
-			(at 80.01 58.42 0)
-			(effects
-				(font
-					(size 1.27 1.27)
-				)
-				(hide yes)
-			)
-		)
-		(pin "1"
-		)
-		(instances
-			(project "CW HF Transceiver"
-				(path "/46807950-96a2-445b-a4f1-43cb63a530a8/3d57e32e-3e27-4526-9430-25edad46b736"
-					(reference "#PWR057")
+					(reference "U6")
 					(unit 1)
 				)
@@
 		(dnp no)
 		(fields_autoplaced yes)
-		(property "Reference" "#PWR059"
+		(property "Reference" "#PWR049"
 			(at 118.11 74.93 0)
 			(effects
@@
 			(project ""
 				(path "/46807950-96a2-445b-a4f1-43cb63a530a8/3d57e32e-3e27-4526-9430-25edad46b736"
-					(reference "#PWR059")
+					(reference "#PWR049")
 					(unit 1)
 				)
@@
 		(dnp no)
 		(fields_autoplaced yes)
-		(property "Reference" "Y3"
+		(property "Reference" "Y2"
 			(at 77.47 115.57 0)
 			(effects
@@
 			(project ""
 				(path "/46807950-96a2-445b-a4f1-43cb63a530a8/3d57e32e-3e27-4526-9430-25edad46b736"
-					(reference "Y3")
+					(reference "Y2")
 					(unit 1)
 				)
@@
 		(dnp no)
 		(fields_autoplaced yes)
-		(property "Reference" "#PWR051"
+		(property "Reference" "#PWR042"
 			(at 39.37 78.74 0)
 			(effects
@@
 			(project ""
 				(path "/46807950-96a2-445b-a4f1-43cb63a530a8/3d57e32e-3e27-4526-9430-25edad46b736"
-					(reference "#PWR051")
+					(reference "#PWR042")
 					(unit 1)
 				)
@@
 		(dnp no)
 		(fields_autoplaced yes)
-		(property "Reference" "C27"
+		(property "Reference" "C20"
 			(at 121.92 63.4999 0)
 			(effects
@@
 			(project ""
 				(path "/46807950-96a2-445b-a4f1-43cb63a530a8/3d57e32e-3e27-4526-9430-25edad46b736"
-					(reference "C27")
+					(reference "C20")
 					(unit 1)
 				)
@@
 		(dnp no)
 		(fields_autoplaced yes)
-		(property "Reference" "#PWR060"
+		(property "Reference" "#PWR050"
 			(at 134.62 115.57 0)
 			(effects
@@
 			(project ""
 				(path "/46807950-96a2-445b-a4f1-43cb63a530a8/3d57e32e-3e27-4526-9430-25edad46b736"
-					(reference "#PWR060")
-					(unit 1)
-				)
+					(reference "#PWR050")
+					(unit 1)
+				)

Commit message: on the final bits!
Parts:
- renumbered C17 to C29, C18 to C30, C19 to C31, C20 to C32, C21 to C33, J5 to J6, R8 to R11, U6 to U7
Changed lines of the file:
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@@
 		(dnp no)
 		(fields_autoplaced yes)
-		(property "Reference" "R8"
+		(property "Reference" "R11"
 			(at 59.69 63.4999 0)
 			(effects
@@
 			(project ""
 				(path "/46807950-96a2-445b-a4f1-43cb63a530a8/3d57e32e-3e27-4526-9430-25edad46b736"
-					(reference "R8")
+					(reference "R11")
 					(unit 1)
 				)
@@
 		(dnp no)
 		(fields_autoplaced yes)
-		(property "Reference" "#PWR047"
+		(property "Reference" "#PWR068"
 			(at 77.47 143.51 0)
 			(effects
@@
 			(project ""
 				(path "/46807950-96a2-445b-a4f1-43cb63a530a8/3d57e32e-3e27-4526-9430-25edad46b736"
-					(reference "#PWR047")
+					(reference "#PWR068")
 					(unit 1)
 				)
@@
 		(dnp no)
 		(fields_autoplaced yes)
-		(property "Reference" "#PWR048"
+		(property "Reference" "#PWR069"
 			(at 95.25 110.49 0)
 			(effects
@@
 			(project ""
 				(path "/46807950-96a2-445b-a4f1-43cb63a530a8/3d57e32e-3e27-4526-9430-25edad46b736"
-					(reference "#PWR048")
+					(reference "#PWR069")
 					(unit 1)
 				)
@@
 		(dnp no)
 		(fields_autoplaced yes)
-		(property "Reference" "#PWR043"
+		(property "Reference" "#PWR064"
 			(at 57.15 64.77 0)
 			(effects
@@
 			(project ""
 				(path "/46807950-96a2-445b-a4f1-43cb63a530a8/3d57e32e-3e27-4526-9430-25edad46b736"
-					(reference "#PWR043")
+					(reference "#PWR064")
 					(unit 1)
 				)
@@
 		(dnp no)
 		(fields_autoplaced yes)
-		(property "Reference" "C21"
+		(property "Reference" "C33"
 			(at 134.62 63.4999 0)
 			(effects
@@
 			(project "CW HF Transceiver"
 				(path "/46807950-96a2-445b-a4f1-43cb63a530a8/3d57e32e-3e27-4526-9430-25edad46b736"
-					(reference "C21")
+					(reference "C33")
 					(unit 1)
 				)
@@
 		(dnp no)
 		(fields_autoplaced yes)
-		(property "Reference" "#PWR044"
+		(property "Reference" "#PWR065"
 			(at 60.96 104.14 0)
 			(effects
@@
 			(project ""
 				(path "/46807950-96a2-445b-a4f1-43cb63a530a8/3d57e32e-3e27-4526-9430-25edad46b736"
-					(reference "#PWR044")
+					(reference "#PWR065")
 					(unit 1)
 				)
@@
 		(dnp no)
 		(fields_autoplaced yes)
-		(property "Reference" "C17"
+		(property "Reference" "C29"
 			(at 72.39 126.9999 0)
 			(effects
@@
 			(project ""
 				(path "/46807950-96a2-445b-a4f1-43cb63a530a8/3d57e32e-3e27-4526-9430-25edad46b736"
-					(reference "C17")
+					(reference "C29")
 					(unit 1)
 				)
@@
 		(dnp no)
 		(fields_autoplaced yes)
-		(property "Reference" "C19"
+		(property "Reference" "C31"
 			(at 105.41 63.4999 0)
 			(effects
@@
 			(project ""
 				(path "/46807950-96a2-445b-a4f1-43cb63a530a8/3d57e32e-3e27-4526-9430-25edad46b736"
-					(reference "C19")
+					(reference "C31")
 					(unit 1)
 				)
@@
 		(dnp no)
 		(fields_autoplaced yes)
-		(property "Reference" "#PWR046"
+		(property "Reference" "#PWR067"
 			(at 77.47 113.03 0)
 			(effects
@@
 			(project "CW HF Transceiver"
 				(path "/46807950-96a2-445b-a4f1-43cb63a530a8/3d57e32e-3e27-4526-9430-25edad46b736"
-					(reference "#PWR046")
+					(reference "#PWR067")
 					(unit 1)
 				)
@@
 		(dnp no)
 		(fields_autoplaced yes)
-		(property "Reference" "C18"
+		(property "Reference" "C30"
 			(at 90.17 126.9999 0)
 			(effects
@@
 			(project "CW HF Transceiver"
 				(path "/46807950-96a2-445b-a4f1-43cb63a530a8/3d57e32e-3e27-4526-9430-25edad46b736"
-					(reference "C18")
+					(reference "C30")
 					(unit 1)
 				)
@@
 		(on_board yes)
 		(dnp no)
-		(property "Reference" "J5"
+		(property "Reference" "J6"
 			(at 147.955 96.52 0)
 			(effects
@@
 			(project ""
 				(path "/46807950-96a2-445b-a4f1-43cb63a530a8/3d57e32e-3e27-4526-9430-25edad46b736"
-					(reference "J5")
+					(reference "J6")
 					(unit 1)
 				)
@@
 		(dnp no)
 		(fields_autoplaced yes)
-		(property "Reference" "#PWR045"
+		(property "Reference" "#PWR066"
 			(at 74.93 62.23 0)
 			(effects
@@
 			(project ""
 				(path "/46807950-96a2-445b-a4f1-43cb63a530a8/3d57e32e-3e27-4526-9430-25edad46b736"
-					(reference "#PWR045")
+					(reference "#PWR066")
 					(unit 1)
 				)
@@
 		(on_board yes)
 		(dnp no)
-		(property "Reference" "U6"
+		(property "Reference" "U7"
 			(at 82.2041 57.15 0)
 			(effects
@@
 			(project ""
 				(path "/46807950-96a2-445b-a4f1-43cb63a530a8/3d57e32e-3e27-4526-9430-25edad46b736"
-					(reference "U6")
+					(reference "U7")
 					(unit 1)
 				)
@@
 		(dnp no)
 		(fields_autoplaced yes)
-		(property "Reference" "#PWR049"
+		(property "Reference" "#PWR070"
 			(at 118.11 74.93 0)
 			(effects
@@
 			(project ""
 				(path "/46807950-96a2-445b-a4f1-43cb63a530a8/3d57e32e-3e27-4526-9430-25edad46b736"
-					(reference "#PWR049")
+					(reference "#PWR070")
 					(unit 1)
 				)
@@
 		(dnp no)
 		(fields_autoplaced yes)
-		(property "Reference" "#PWR042"
+		(property "Reference" "#PWR063"
 			(at 39.37 78.74 0)
 			(effects
@@
 			(project ""
 				(path "/46807950-96a2-445b-a4f1-43cb63a530a8/3d57e32e-3e27-4526-9430-25edad46b736"
-					(reference "#PWR042")
+					(reference "#PWR063")
 					(unit 1)
 				)
@@
 		(dnp no)
 		(fields_autoplaced yes)
-		(property "Reference" "C20"
+		(property "Reference" "C32"
 			(at 121.92 63.4999 0)
 			(effects
@@
 			(project ""
 				(path "/46807950-96a2-445b-a4f1-43cb63a530a8/3d57e32e-3e27-4526-9430-25edad46b736"
-					(reference "C20")
+					(reference "C32")
 					(unit 1)
 				)
@@
 		(dnp no)
 		(fields_autoplaced yes)
-		(property "Reference" "#PWR050"
+		(property "Reference" "#PWR071"
 			(at 134.62 115.57 0)
 			(effects
@@
 			(project ""
 				(path "/46807950-96a2-445b-a4f1-43cb63a530a8/3d57e32e-3e27-4526-9430-25edad46b736"
-					(reference "#PWR050")
-					(unit 1)
-				)
+					(reference "#PWR071")
+					(unit 1)
+				)

Commit message: should be done
Parts:
- renumbered C29 to C30, C30 to C31, C31 to C32, C32 to C33, C33 to C34, J6 to J7, SW2 to SW1
Connections:
- net Input to receiver renamed Input
Changed lines of the file:
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@@
 		)
 	)
-	(hierarchical_label "Input to receiver"
+	(hierarchical_label "Input"
 		(shape input)
 		(at 96.52 88.9 0)
@@
 		(dnp no)
 		(fields_autoplaced yes)
-		(property "Reference" "#PWR068"
+		(property "Reference" "#PWR069"
 			(at 77.47 143.51 0)
 			(effects
@@
 			(project ""
 				(path "/46807950-96a2-445b-a4f1-43cb63a530a8/3d57e32e-3e27-4526-9430-25edad46b736"
-					(reference "#PWR068")
+					(reference "#PWR069")
 					(unit 1)
 				)
@@
 		(dnp no)
 		(fields_autoplaced yes)
-		(property "Reference" "#PWR069"
+		(property "Reference" "#PWR070"
 			(at 95.25 110.49 0)
 			(effects
@@
 			(project ""
 				(path "/46807950-96a2-445b-a4f1-43cb63a530a8/3d57e32e-3e27-4526-9430-25edad46b736"
-					(reference "#PWR069")
+					(reference "#PWR070")
 					(unit 1)
 				)
@@
 		(dnp no)
 		(fields_autoplaced yes)
-		(property "Reference" "#PWR064"
+		(property "Reference" "#PWR065"
 			(at 57.15 64.77 0)
 			(effects
@@
 			(project ""
 				(path "/46807950-96a2-445b-a4f1-43cb63a530a8/3d57e32e-3e27-4526-9430-25edad46b736"
-					(reference "#PWR064")
+					(reference "#PWR065")
 					(unit 1)
 				)
@@
 		(dnp no)
 		(fields_autoplaced yes)
-		(property "Reference" "C33"
+		(property "Reference" "C34"
 			(at 134.62 63.4999 0)
 			(effects
@@
 			(project "CW HF Transceiver"
 				(path "/46807950-96a2-445b-a4f1-43cb63a530a8/3d57e32e-3e27-4526-9430-25edad46b736"
-					(reference "C33")
+					(reference "C34")
 					(unit 1)
 				)
@@
 		(dnp no)
 		(fields_autoplaced yes)
-		(property "Reference" "#PWR065"
+		(property "Reference" "#PWR066"
 			(at 60.96 104.14 0)
 			(effects
@@
 			(project ""
 				(path "/46807950-96a2-445b-a4f1-43cb63a530a8/3d57e32e-3e27-4526-9430-25edad46b736"
-					(reference "#PWR065")
+					(reference "#PWR066")
 					(unit 1)
 				)
@@
 		(dnp no)
 		(fields_autoplaced yes)
-		(property "Reference" "C29"
+		(property "Reference" "C30"
 			(at 72.39 126.9999 0)
 			(effects
@@
 			(project ""
 				(path "/46807950-96a2-445b-a4f1-43cb63a530a8/3d57e32e-3e27-4526-9430-25edad46b736"
-					(reference "C29")
+					(reference "C30")
 					(unit 1)
 				)
@@
 		(dnp no)
 		(fields_autoplaced yes)
-		(property "Reference" "SW2"
+		(property "Reference" "SW1"
 			(at 48.26 63.5 0)
 			(effects
@@
 			(project ""
 				(path "/46807950-96a2-445b-a4f1-43cb63a530a8/3d57e32e-3e27-4526-9430-25edad46b736"
-					(reference "SW2")
+					(reference "SW1")
 					(unit 1)
 				)
@@
 		(dnp no)
 		(fields_autoplaced yes)
-		(property "Reference" "C31"
+		(property "Reference" "C32"
 			(at 105.41 63.4999 0)
 			(effects
@@
 			(project ""
 				(path "/46807950-96a2-445b-a4f1-43cb63a530a8/3d57e32e-3e27-4526-9430-25edad46b736"
-					(reference "C31")
+					(reference "C32")
 					(unit 1)
 				)
@@
 		(dnp no)
 		(fields_autoplaced yes)
-		(property "Reference" "#PWR067"
+		(property "Reference" "#PWR068"
 			(at 77.47 113.03 0)
 			(effects
@@
 			(project "CW HF Transceiver"
 				(path "/46807950-96a2-445b-a4f1-43cb63a530a8/3d57e32e-3e27-4526-9430-25edad46b736"
-					(reference "#PWR067")
+					(reference "#PWR068")
 					(unit 1)
 				)
@@
 		(dnp no)
 		(fields_autoplaced yes)
-		(property "Reference" "C30"
+		(property "Reference" "C31"
 			(at 90.17 126.9999 0)
 			(effects
@@
 			(project "CW HF Transceiver"
 				(path "/46807950-96a2-445b-a4f1-43cb63a530a8/3d57e32e-3e27-4526-9430-25edad46b736"
-					(reference "C30")
+					(reference "C31")
 					(unit 1)
 				)
@@
 		(on_board yes)
 		(dnp no)
-		(property "Reference" "J6"
+		(property "Reference" "J7"
 			(at 147.955 96.52 0)
 			(effects
@@
 			(project ""
 				(path "/46807950-96a2-445b-a4f1-43cb63a530a8/3d57e32e-3e27-4526-9430-25edad46b736"
-					(reference "J6")
+					(reference "J7")
 					(unit 1)
 				)
@@
 		(dnp no)
 		(fields_autoplaced yes)
-		(property "Reference" "#PWR066"
+		(property "Reference" "#PWR067"
 			(at 74.93 62.23 0)
 			(effects
@@
 			(project ""
 				(path "/46807950-96a2-445b-a4f1-43cb63a530a8/3d57e32e-3e27-4526-9430-25edad46b736"
-					(reference "#PWR066")
+					(reference "#PWR067")
 					(unit 1)
 				)
@@
 		(dnp no)
 		(fields_autoplaced yes)
-		(property "Reference" "#PWR070"
+		(property "Reference" "#PWR071"
 			(at 118.11 74.93 0)
 			(effects
@@
 			(project ""
 				(path "/46807950-96a2-445b-a4f1-43cb63a530a8/3d57e32e-3e27-4526-9430-25edad46b736"
-					(reference "#PWR070")
+					(reference "#PWR071")
 					(unit 1)
 				)
@@
 		(dnp no)
 		(fields_autoplaced yes)
-		(property "Reference" "#PWR063"
+		(property "Reference" "#PWR064"
 			(at 39.37 78.74 0)
 			(effects
@@
 			(project ""
 				(path "/46807950-96a2-445b-a4f1-43cb63a530a8/3d57e32e-3e27-4526-9430-25edad46b736"
-					(reference "#PWR063")
+					(reference "#PWR064")
 					(unit 1)
 				)
@@
 		(dnp no)
 		(fields_autoplaced yes)
-		(property "Reference" "C32"
+		(property "Reference" "C33"
 			(at 121.92 63.4999 0)
 			(effects
@@
 			(project ""
 				(path "/46807950-96a2-445b-a4f1-43cb63a530a8/3d57e32e-3e27-4526-9430-25edad46b736"
-					(reference "C32")
+					(reference "C33")
 					(unit 1)
 				)
@@
 		(dnp no)
 		(fields_autoplaced yes)
-		(property "Reference" "#PWR071"
+		(property "Reference" "#PWR072"
 			(at 134.62 115.57 0)
 			(effects
@@
 			(project ""
 				(path "/46807950-96a2-445b-a4f1-43cb63a530a8/3d57e32e-3e27-4526-9430-25edad46b736"
-					(reference "#PWR071")
-					(unit 1)
-				)
+					(reference "#PWR072")
+					(unit 1)
+				)

Commit message: add the pcb
Parts:
- removed C30, C31: 22p, Capacitor_SMD:C_0603_1608Metric, symbol Device:C
- removed J7: AudioJack3, symbol Connector_Audio:AudioJack3
- removed SW1: Reset RX, symbol Switch:SW_Push
- removed Y2: 37.628KHz, symbol Device:Crystal
- added Audio2: PJ-327C-4A, plib:AUDIO-SMD_PJ-327C-4A, symbol plib:PJ-327C-4A
- added JP1: RST RX, Jumper:SolderJumper-2_P1.3mm_Open_RoundedPad1.0x1.5mm, symbol Jumper:SolderJumper_2_Open
- U7: footprint (none) -> Package_SO:SSOP-24_3.9x8.7mm_P0.635mm
- renumbered C32 to C29, C33 to C30, C34 to C31
Connections:
- net GND: now also Audio2.1, JP1.1 (A)
- net Lout: now also Audio2.2
- net Rout: now also Audio2.3
- net at R11.2, U7.15 (~{RST}): now also JP1.2 (B)
- net DCLK: no longer names the net of U7.3 (GPO3/[DCLK])
- net RCLK renamed Receiver clk
- no-connect marks 4 -> 6
