File: VFO.kicad_sch (KiCad schematic)
At the start: 4 parts, among them U5 Si5351A-B-GT, Y1 25MHz

Commit message: a
Connections:
- net GND: no longer U5.9 (CLK1)
- new net tune out: U5.9 (CLK1)
Changed lines of the file:
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@@
 	(generator_version "8.0")
 	(paper "A4")
-	(junction
-		(at 153.67 90.17)
-		(diameter 0)
-		(color 0 0 0 0)
-	)
 	(wire
 		(pts
 			(xy 124.46 76.2) (xy 124.46 77.47)
-		)
-		(stroke
-			(width 0)
-			(type default)
-		)
-	)
-	(wire
-		(pts
-			(xy 153.67 85.09) (xy 153.67 90.17)
 		)
 		(stroke
@@
 	(wire
 		(pts
-			(xy 152.4 85.09) (xy 153.67 85.09)
+			(xy 152.4 85.09) (xy 154.94 85.09)
 		)
 		(stroke
@@
 		)
 	)
+	(hierarchical_label "tune out"
+		(shape output)
+		(at 154.94 85.09 0)
+		(fields_autoplaced yes)
+		(effects
+			(font
+				(size 1.27 1.27)
+			)
+			(justify left)
+		)
+	)

Commit message: update
Connections:
- net +3.3V: now also U5.7 (VDDO)
- net VCC: no longer U5.7 (VDDO)
Changed lines of the file:
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@@
 	(generator_version "8.0")
 	(paper "A4")
+	(junction
+		(at 137.16 69.85)
+		(diameter 0)
+		(color 0 0 0 0)
+	)
 	(wire
 		(pts
@@
 	(wire
 		(pts
+			(xy 137.16 69.85) (xy 137.16 72.39)
+		)
+		(stroke
+			(width 0)
+			(type default)
+		)
+	)
+	(wire
+		(pts
 			(xy 152.4 90.17) (xy 153.67 90.17)
 		)
@@
 	(wire
 		(pts
+			(xy 124.46 77.47) (xy 127 77.47)
+		)
+		(stroke
+			(width 0)
+			(type default)
+		)
+	)
+	(wire
+		(pts
+			(xy 120.65 83.82) (xy 124.46 83.82)
+		)
+		(stroke
+			(width 0)
+			(type default)
+		)
+	)
+	(wire
+		(pts
+			(xy 125.73 92.71) (xy 127 92.71)
+		)
+		(stroke
+			(width 0)
+			(type default)
+		)
+	)
+	(wire
+		(pts
+			(xy 142.24 69.85) (xy 137.16 69.85)
+		)
+		(stroke
+			(width 0)
+			(type default)
+		)
+	)
+	(wire
+		(pts
+			(xy 124.46 83.82) (xy 124.46 82.55)
+		)
+		(stroke
+			(width 0)
+			(type default)
+		)
+	)
+	(wire
+		(pts
+			(xy 125.73 90.17) (xy 127 90.17)
+		)
+		(stroke
+			(width 0)
+			(type default)
+		)
+	)
+	(wire
+		(pts
+			(xy 152.4 80.01) (xy 154.94 80.01)
+		)
+		(stroke
+			(width 0)
+			(type default)
+		)
+	)
+	(wire
+		(pts
+			(xy 137.16 69.85) (xy 137.16 68.58)
+		)
+		(stroke
+			(width 0)
+			(type default)
+		)
+	)
+	(wire
+		(pts
+			(xy 152.4 85.09) (xy 154.94 85.09)
+		)
+		(stroke
+			(width 0)
+			(type default)
+		)
+	)
+	(wire
+		(pts
 			(xy 120.65 76.2) (xy 124.46 76.2)
 		)
@@
 	(wire
 		(pts
-			(xy 124.46 77.47) (xy 127 77.47)
-		)
-		(stroke
-			(width 0)
-			(type default)
-		)
-	)
-	(wire
-		(pts
-			(xy 120.65 83.82) (xy 124.46 83.82)
-		)
-		(stroke
-			(width 0)
-			(type default)
-		)
-	)
-	(wire
-		(pts
-			(xy 125.73 92.71) (xy 127 92.71)
-		)
-		(stroke
-			(width 0)
-			(type default)
-		)
-	)
-	(wire
-		(pts
-			(xy 124.46 83.82) (xy 124.46 82.55)
-		)
-		(stroke
-			(width 0)
-			(type default)
-		)
-	)
-	(wire
-		(pts
-			(xy 125.73 90.17) (xy 127 90.17)
-		)
-		(stroke
-			(width 0)
-			(type default)
-		)
-	)
-	(wire
-		(pts
-			(xy 152.4 80.01) (xy 154.94 80.01)
-		)
-		(stroke
-			(width 0)
-			(type default)
-		)
-	)
-	(wire
-		(pts
-			(xy 152.4 85.09) (xy 154.94 85.09)
+			(xy 142.24 72.39) (xy 142.24 69.85)
 		)
 		(stroke
@@
 	(symbol
 		(lib_id "power:+3.3V")
-		(at 137.16 72.39 0)
+		(at 137.16 68.58 0)
 		(unit 1)
 		(exclude_from_sim no)
@@
 		(fields_autoplaced yes)
 		(property "Reference" "#PWR01"
-			(at 137.16 76.2 0)
+			(at 137.16 72.39 0)
 			(effects
 				(font
@@
 		)
 		(property "Value" "+3.3V"
-			(at 137.16 67.31 0)
+			(at 137.16 63.5 0)
 			(effects
 				(font
@@
 		)
 		(property "Footprint" ""
-			(at 137.16 72.39 0)
+			(at 137.16 68.58 0)
 			(effects
 				(font
@@
 		)
 		(property "Datasheet" ""
-			(at 137.16 72.39 0)
+			(at 137.16 68.58 0)
 			(effects
 				(font
@@
 		)
 		(property "Description" "Power symbol creates a global label with name \"+3.3V\""
-			(at 137.16 72.39 0)
+			(at 137.16 68.58 0)
 			(effects
 				(font
@@
 					(unit 1)
 				)
-			)
-		)
-	)
-	(symbol
-		(lib_id "power:VCC")
-		(at 142.24 72.39 0)
-		(unit 1)
-		(exclude_from_sim no)
-		(in_bom yes)
-		(on_board yes)
-		(dnp no)
-		(fields_autoplaced yes)
-		(property "Reference" "#PWR020"
-			(at 142.24 76.2 0)
-			(effects
-				(font
-					(size 1.27 1.27)
-				)
-				(hide yes)
-			)
-		)
-		(property "Value" "VCC"
-			(at 142.24 67.31 0)
-			(effects
-				(font
-					(size 1.27 1.27)
-				)
-			)
-		)
-		(property "Footprint" ""
-			(at 142.24 72.39 0)
-			(effects
-				(font
-					(size 1.27 1.27)
-				)
-				(hide yes)
-			)
-		)
-		(property "Datasheet" ""
-			(at 142.24 72.39 0)
-			(effects
-				(font
-					(size 1.27 1.27)
-				)
-				(hide yes)
-			)
-		)
-		(property "Description" "Power symbol creates a global label with name \"VCC\""
-			(at 142.24 72.39 0)
-			(effects
-				(font
-					(size 1.27 1.27)
-				)
-				(hide yes)
-			)
-		)
-		(pin "1"
-		)
-		(instances
-			(project "CW HF Transceiver"
-				(path "/46807950-96a2-445b-a4f1-43cb63a530a8/7a390537-499b-4027-b8ee-d9509676514b"
-					(reference "#PWR020")
-					(unit 1)
-				)

Commit message: Update amp
Parts:
- added TP2, TP3: TestPoint, symbol Connector:TestPoint
Connections:
- net tune out: now also TP3.1
- net wave out: now also TP2.1
Changed lines of the file:
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@@
 	(paper "A4")
+	(junction
+		(at 153.67 85.09)
+		(diameter 0)
+		(color 0 0 0 0)
+	)
 	(junction
 		(at 137.16 69.85)
@@
 		(color 0 0 0 0)
 	)
+	(junction
+		(at 153.67 80.01)
+		(diameter 0)
+		(color 0 0 0 0)
+	)
 	(wire
 		(pts
@@
 	(wire
 		(pts
-			(xy 152.4 80.01) (xy 154.94 80.01)
+			(xy 153.67 85.09) (xy 154.94 85.09)
+		)
+		(stroke
+			(width 0)
+			(type default)
+		)
+	)
+	(wire
+		(pts
+			(xy 152.4 80.01) (xy 153.67 80.01)
 		)
 		(stroke
@@
 	(wire
 		(pts
-			(xy 152.4 85.09) (xy 154.94 85.09)
+			(xy 152.4 85.09) (xy 153.67 85.09)
 		)
 		(stroke
@@
 		(pts
 			(xy 153.67 90.17) (xy 153.67 92.71)
+		)
+		(stroke
+			(width 0)
+			(type default)
+		)
+	)
+	(wire
+		(pts
+			(xy 153.67 80.01) (xy 154.94 80.01)
 		)
 		(stroke
@@
 					(unit 1)
 				)
+			)
+		)
+	)
+	(symbol
+		(lib_id "Connector:TestPoint")
+		(at 153.67 85.09 180)
+		(unit 1)
+		(exclude_from_sim no)
+		(in_bom yes)
+		(on_board yes)
+		(dnp no)
+		(fields_autoplaced yes)
+		(property "Reference" "TP3"
+			(at 156.21 87.1219 0)
+			(effects
+				(font
+					(size 1.27 1.27)
+				)
+				(justify right)
+			)
+		)
+		(property "Value" "TestPoint"
+			(at 156.21 89.6619 0)
+			(effects
+				(font
+					(size 1.27 1.27)
+				)
+				(justify right)
+			)
+		)
+		(property "Footprint" ""
+			(at 148.59 85.09 0)
+			(effects
+				(font
+					(size 1.27 1.27)
+				)
+				(hide yes)
+			)
+		)
+		(property "Datasheet" "~"
+			(at 148.59 85.09 0)
+			(effects
+				(font
+					(size 1.27 1.27)
+				)
+				(hide yes)
+			)
+		)
+		(property "Description" "test point"
+			(at 153.67 85.09 0)
+			(effects
+				(font
+					(size 1.27 1.27)
+				)
+				(hide yes)
+			)
+		)
+		(pin "1"
+		)
+		(instances
+			(project "CW HF Transceiver"
+				(path "/46807950-96a2-445b-a4f1-43cb63a530a8/7a390537-499b-4027-b8ee-d9509676514b"
+					(reference "TP3")
+					(unit 1)
+				)
+			)
+		)
+	)
+	(symbol
+		(lib_id "Connector:TestPoint")
+		(at 153.67 80.01 0)
+		(unit 1)
+		(exclude_from_sim no)
+		(in_bom yes)
+		(on_board yes)
+		(dnp no)
+		(fields_autoplaced yes)
+		(property "Reference" "TP2"
+			(at 156.21 75.4379 0)
+			(effects
+				(font
+					(size 1.27 1.27)
+				)
+				(justify left)
+			)
+		)
+		(property "Value" "TestPoint"
+			(at 156.21 77.9779 0)
+			(effects
+				(font
+					(size 1.27 1.27)
+				)
+				(justify left)
+			)
+		)
+		(property "Footprint" ""
+			(at 158.75 80.01 0)
+			(effects
+				(font
+					(size 1.27 1.27)
+				)
+				(hide yes)
+			)
+		)
+		(property "Datasheet" "~"
+			(at 158.75 80.01 0)
+			(effects
+				(font
+					(size 1.27 1.27)
+				)
+				(hide yes)
+			)
+		)
+		(property "Description" "test point"
+			(at 153.67 80.01 0)
+			(effects
+				(font
+					(size 1.27 1.27)
+				)
+				(hide yes)
+			)
+		)
+		(pin "1"
+		)
+		(instances
+			(project "CW HF Transceiver"
+				(path "/46807950-96a2-445b-a4f1-43cb63a530a8/7a390537-499b-4027-b8ee-d9509676514b"
+					(reference "TP2")
+					(unit 1)
+				)

Commit message: some big updates
Parts:
- added TP4: CLK2, symbol Connector:TestPoint
- C19: renamed from C15; value 1uF -> 1u; footprint (none) -> Capacitor_SMD:C_0603_1608Metric
- C20: renamed from C16; value 1uF -> 1u; footprint (none) -> Capacitor_SMD:C_0603_1608Metric
- TP3: renamed from TP2; value TestPoint -> CLK0
- TP5: renamed from TP3; value TestPoint -> CLK1
- U4: renamed from U5; footprint Package_SO:MSOP-10_3x3mm_P0.5mm -> (none)
- Y2: renamed from Y1; footprint Crystal:Crystal_AT310_D3.0mm_L10.0mm_Horizontal -> (none)
Connections:
- net GND: no longer U4.6 (CLK2)
- net tune out renamed 180º Wave Out
- net wave out renamed Wave out
- new net BFO out: TP4.1, U4.6 (CLK2)
Other:
- title: (none) -> Si5351a Controller
- moved on the sheet: C19, C20, TP5

Commit message: update
Parts:
- added C10, C11: 10p, symbol Device:C
- U3: renamed from U4; footprint (none) -> Package_SO:MSOP-10_3x3mm_P0.5mm
- renumbered C19 to C12, C20 to C13, TP3 to TP4, TP4 to TP5, TP5 to TP6, Y2 to Y1
Connections:
- net GND: now also C10.1, C11.1
- net at U3.2 (XA), Y1.1: now also C10.2
- net at U3.3 (XB), Y1.2: now also C11.2

Commit message: on the final bits!
Parts:
- renumbered C10 to C21, C11 to C22, C12 to C23, C13 to C24, TP4 to TP3, TP5 to TP4, TP6 to TP5, U3 to U4
Changed lines of the file:
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@@
 		(dnp no)
 		(fields_autoplaced yes)
-		(property "Reference" "#PWR026"
+		(property "Reference" "#PWR045"
 			(at 137.16 72.39 0)
 			(effects
@@
 			(project "CW HF Transceiver"
 				(path "/46807950-96a2-445b-a4f1-43cb63a530a8/7a390537-499b-4027-b8ee-d9509676514b"
-					(reference "#PWR026")
+					(reference "#PWR045")
 					(unit 1)
 				)
@@
 		(on_board yes)
 		(dnp no)
-		(property "Reference" "TP6"
+		(property "Reference" "TP5"
 			(at 168.91 87.1219 0)
 			(effects
@@
 			(project "CW HF Transceiver"
 				(path "/46807950-96a2-445b-a4f1-43cb63a530a8/7a390537-499b-4027-b8ee-d9509676514b"
-					(reference "TP6")
+					(reference "TP5")
 					(unit 1)
 				)
@@
 		(dnp no)
 		(fields_autoplaced yes)
-		(property "Reference" "#PWR025"
+		(property "Reference" "#PWR044"
 			(at 95.25 92.71 0)
 			(effects
@@
 			(project ""
 				(path "/46807950-96a2-445b-a4f1-43cb63a530a8/7a390537-499b-4027-b8ee-d9509676514b"
-					(reference "#PWR025")
+					(reference "#PWR044")
 					(unit 1)
 				)
@@
 		(dnp no)
 		(fields_autoplaced yes)
-		(property "Reference" "TP4"
+		(property "Reference" "TP3"
 			(at 156.21 75.4379 0)
 			(effects
@@
 			(project "CW HF Transceiver"
 				(path "/46807950-96a2-445b-a4f1-43cb63a530a8/7a390537-499b-4027-b8ee-d9509676514b"
-					(reference "TP4")
+					(reference "TP3")
 					(unit 1)
 				)
@@
 		(dnp no)
 		(fields_autoplaced yes)
-		(property "Reference" "C10"
+		(property "Reference" "C21"
 			(at 100.33 68.58 90)
 			(effects
@@
 			(project ""
 				(path "/46807950-96a2-445b-a4f1-43cb63a530a8/7a390537-499b-4027-b8ee-d9509676514b"
-					(reference "C10")
+					(reference "C21")
 					(unit 1)
 				)
@@
 		(dnp no)
 		(fields_autoplaced yes)
-		(property "Reference" "#PWR027"
+		(property "Reference" "#PWR046"
 			(at 139.7 104.14 0)
 			(effects
@@
 			(project "CW HF Transceiver"
 				(path "/46807950-96a2-445b-a4f1-43cb63a530a8/7a390537-499b-4027-b8ee-d9509676514b"
-					(reference "#PWR027")
+					(reference "#PWR046")
 					(unit 1)
 				)
@@
 		(dnp no)
 		(fields_autoplaced yes)
-		(property "Reference" "#PWR030"
+		(property "Reference" "#PWR049"
 			(at 209.55 86.36 0)
 			(effects
@@
 			(project "CW HF Transceiver"
 				(path "/46807950-96a2-445b-a4f1-43cb63a530a8/7a390537-499b-4027-b8ee-d9509676514b"
-					(reference "#PWR030")
+					(reference "#PWR049")
 					(unit 1)
 				)
@@
 		(dnp no)
 		(fields_autoplaced yes)
-		(property "Reference" "U3"
+		(property "Reference" "U4"
 			(at 141.8941 97.79 0)
 			(effects
@@
 			(project "CW HF Transceiver"
 				(path "/46807950-96a2-445b-a4f1-43cb63a530a8/7a390537-499b-4027-b8ee-d9509676514b"
-					(reference "U3")
+					(reference "U4")
 					(unit 1)
 				)
@@
 		(dnp no)
 		(fields_autoplaced yes)
-		(property "Reference" "#PWR031"
+		(property "Reference" "#PWR050"
 			(at 209.55 96.52 0)
 			(effects
@@
 			(project "CW HF Transceiver"
 				(path "/46807950-96a2-445b-a4f1-43cb63a530a8/7a390537-499b-4027-b8ee-d9509676514b"
-					(reference "#PWR031")
+					(reference "#PWR050")
 					(unit 1)
 				)
@@
 		(on_board yes)
 		(dnp no)
-		(property "Reference" "C11"
+		(property "Reference" "C22"
 			(at 100.33 80.264 90)
 			(effects
@@
 			(project "CW HF Transceiver"
 				(path "/46807950-96a2-445b-a4f1-43cb63a530a8/7a390537-499b-4027-b8ee-d9509676514b"
-					(reference "C11")
+					(reference "C22")
 					(unit 1)
 				)
@@
 		(dnp no)
 		(fields_autoplaced yes)
-		(property "Reference" "#PWR028"
+		(property "Reference" "#PWR047"
 			(at 196.85 86.36 0)
 			(effects
@@
 			(project "CW HF Transceiver"
 				(path "/46807950-96a2-445b-a4f1-43cb63a530a8/7a390537-499b-4027-b8ee-d9509676514b"
-					(reference "#PWR028")
+					(reference "#PWR047")
 					(unit 1)
 				)
@@
 		(dnp no)
 		(fields_autoplaced yes)
-		(property "Reference" "TP5"
+		(property "Reference" "TP4"
 			(at 161.29 96.0119 0)
 			(effects
@@
 			(project "CW HF Transceiver"
 				(path "/46807950-96a2-445b-a4f1-43cb63a530a8/7a390537-499b-4027-b8ee-d9509676514b"
-					(reference "TP5")
+					(reference "TP4")
 					(unit 1)
 				)
@@
 		(dnp no)
 		(fields_autoplaced yes)
-		(property "Reference" "C13"
+		(property "Reference" "C24"
 			(at 213.36 85.0899 0)
 			(effects
@@
 			(project "CW HF Transceiver"
 				(path "/46807950-96a2-445b-a4f1-43cb63a530a8/7a390537-499b-4027-b8ee-d9509676514b"
-					(reference "C13")
+					(reference "C24")
 					(unit 1)
 				)
@@
 		(dnp no)
 		(fields_autoplaced yes)
-		(property "Reference" "#PWR029"
+		(property "Reference" "#PWR048"
 			(at 196.85 96.52 0)
 			(effects
@@
 			(project "CW HF Transceiver"
 				(path "/46807950-96a2-445b-a4f1-43cb63a530a8/7a390537-499b-4027-b8ee-d9509676514b"
-					(reference "#PWR029")
+					(reference "#PWR048")
 					(unit 1)
 				)
@@
 		(dnp no)
 		(fields_autoplaced yes)
-		(property "Reference" "C12"
+		(property "Reference" "C23"
 			(at 200.66 85.0899 0)
 			(effects
@@
 			(project "CW HF Transceiver"
 				(path "/46807950-96a2-445b-a4f1-43cb63a530a8/7a390537-499b-4027-b8ee-d9509676514b"
-					(reference "C12")
-					(unit 1)
-				)
+					(reference "C23")
+					(unit 1)
+				)

Commit message: should be done
Parts:
- renumbered C21 to C22, C22 to C23, C23 to C24, C24 to C25
Connections:
- net BFO out: no longer names the net of TP4.1, U4.6 (CLK2)
Changed lines of the file:
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@@
-	)
-	(junction
-		(at 158.75 93.98)
-		(diameter 0)
-		(color 0 0 0 0)
 	)
 	(junction
@@
 	(wire
 		(pts
-			(xy 158.75 93.98) (xy 162.56 93.98)
-		)
-		(stroke
-			(width 0)
-			(type default)
-		)
-	)
-	(wire
-		(pts
 			(xy 137.16 69.85) (xy 137.16 72.39)
 		)
@@
 		)
 	)
-	(hierarchical_label "BFO out"
+	(hierarchical_label "180º Wave Out"
 		(shape output)
-		(at 162.56 93.98 0)
+		(at 167.64 85.09 0)
 		(fields_autoplaced yes)
 		(effects
@@
 		)
 	)
-	(hierarchical_label "180º Wave Out"
+	(hierarchical_label "Wave out"
 		(shape output)
-		(at 167.64 85.09 0)
+		(at 154.94 80.01 0)
 		(fields_autoplaced yes)
 		(effects
@@
 		)
 	)
-	(hierarchical_label "Wave out"
-		(shape output)
-		(at 154.94 80.01 0)
-		(fields_autoplaced yes)
-		(effects
-			(font
-				(size 1.27 1.27)
-			)
-			(justify left)
-		)
-	)
 	(symbol
 		(lib_id "power:+3.3V")
@@
 		(dnp no)
 		(fields_autoplaced yes)
-		(property "Reference" "#PWR045"
+		(property "Reference" "#PWR047"
 			(at 137.16 72.39 0)
 			(effects
@@
 			(project "CW HF Transceiver"
 				(path "/46807950-96a2-445b-a4f1-43cb63a530a8/7a390537-499b-4027-b8ee-d9509676514b"
-					(reference "#PWR045")
+					(reference "#PWR047")
 					(unit 1)
 				)
@@
 		(dnp no)
 		(fields_autoplaced yes)
-		(property "Reference" "#PWR044"
+		(property "Reference" "#PWR046"
 			(at 95.25 92.71 0)
 			(effects
@@
 			(project ""
 				(path "/46807950-96a2-445b-a4f1-43cb63a530a8/7a390537-499b-4027-b8ee-d9509676514b"
-					(reference "#PWR044")
+					(reference "#PWR046")
 					(unit 1)
 				)
@@
 		(dnp no)
 		(fields_autoplaced yes)
-		(property "Reference" "C21"
+		(property "Reference" "C22"
 			(at 100.33 68.58 90)
 			(effects
@@
 			(project ""
 				(path "/46807950-96a2-445b-a4f1-43cb63a530a8/7a390537-499b-4027-b8ee-d9509676514b"
-					(reference "C21")
+					(reference "C22")
 					(unit 1)
 				)
@@
 		(dnp no)
 		(fields_autoplaced yes)
-		(property "Reference" "#PWR046"
+		(property "Reference" "#PWR048"
 			(at 139.7 104.14 0)
 			(effects
@@
 			(project "CW HF Transceiver"
 				(path "/46807950-96a2-445b-a4f1-43cb63a530a8/7a390537-499b-4027-b8ee-d9509676514b"
-					(reference "#PWR046")
+					(reference "#PWR048")
 					(unit 1)
 				)
@@
 		(dnp no)
 		(fields_autoplaced yes)
-		(property "Reference" "#PWR049"
+		(property "Reference" "#PWR051"
 			(at 209.55 86.36 0)
 			(effects
@@
 			(project "CW HF Transceiver"
 				(path "/46807950-96a2-445b-a4f1-43cb63a530a8/7a390537-499b-4027-b8ee-d9509676514b"
-					(reference "#PWR049")
+					(reference "#PWR051")
 					(unit 1)
 				)
@@
 		(dnp no)
 		(fields_autoplaced yes)
-		(property "Reference" "#PWR050"
+		(property "Reference" "#PWR052"
 			(at 209.55 96.52 0)
 			(effects
@@
 			(project "CW HF Transceiver"
 				(path "/46807950-96a2-445b-a4f1-43cb63a530a8/7a390537-499b-4027-b8ee-d9509676514b"
-					(reference "#PWR050")
+					(reference "#PWR052")
 					(unit 1)
 				)
@@
 		(on_board yes)
 		(dnp no)
-		(property "Reference" "C22"
+		(property "Reference" "C23"
 			(at 100.33 80.264 90)
 			(effects
@@
 			(project "CW HF Transceiver"
 				(path "/46807950-96a2-445b-a4f1-43cb63a530a8/7a390537-499b-4027-b8ee-d9509676514b"
-					(reference "C22")
+					(reference "C23")
 					(unit 1)
 				)
@@
 		(dnp no)
 		(fields_autoplaced yes)
-		(property "Reference" "#PWR047"
+		(property "Reference" "#PWR049"
 			(at 196.85 86.36 0)
 			(effects
@@
 			(project "CW HF Transceiver"
 				(path "/46807950-96a2-445b-a4f1-43cb63a530a8/7a390537-499b-4027-b8ee-d9509676514b"
-					(reference "#PWR047")
+					(reference "#PWR049")
 					(unit 1)
 				)
@@
 		(dnp no)
 		(fields_autoplaced yes)
-		(property "Reference" "C24"
+		(property "Reference" "C25"
 			(at 213.36 85.0899 0)
 			(effects
@@
 			(project "CW HF Transceiver"
 				(path "/46807950-96a2-445b-a4f1-43cb63a530a8/7a390537-499b-4027-b8ee-d9509676514b"
-					(reference "C24")
+					(reference "C25")
 					(unit 1)
 				)
@@
 		(dnp no)
 		(fields_autoplaced yes)
-		(property "Reference" "#PWR048"
+		(property "Reference" "#PWR050"
 			(at 196.85 96.52 0)
 			(effects
@@
 			(project "CW HF Transceiver"
 				(path "/46807950-96a2-445b-a4f1-43cb63a530a8/7a390537-499b-4027-b8ee-d9509676514b"
-					(reference "#PWR048")
+					(reference "#PWR050")
 					(unit 1)
 				)
@@
 		(dnp no)
 		(fields_autoplaced yes)
-		(property "Reference" "C23"
+		(property "Reference" "C24"
 			(at 200.66 85.0899 0)
 			(effects
@@
 			(project "CW HF Transceiver"
 				(path "/46807950-96a2-445b-a4f1-43cb63a530a8/7a390537-499b-4027-b8ee-d9509676514b"
-					(reference "C23")
-					(unit 1)
-				)
+					(reference "C24")
+					(unit 1)
+				)

Commit message: add the pcb
Parts:
- removed C22, C23: 10p, symbol Device:C
- removed Y1: 25MHz, symbol Device:Crystal
- added Y1: NX3225GA-25.000M-STD-CRG-2, Crystal:Crystal_SMD_3225-4Pin_3.2x2.5mm, symbol Device:Crystal_GND24
- TP2: renamed from TP3; footprint (none) -> TestPoint:TestPoint_Pad_D2.0mm
- TP3: renamed from TP4; footprint (none) -> TestPoint:TestPoint_Pad_D2.0mm
- TP4: renamed from TP5; footprint (none) -> TestPoint:TestPoint_Pad_D2.0mm
- renumbered C24 to C23, C25 to C24
Connections:
- net VCC is gone; now on net +3.3V: C24.1
- net GND: now also Y1.2, Y1.4
- net at U4.2 (XA): now also Y1.3
- net at U4.3 (XB): now also Y1.1
- net Receiver clk: now reaches TP3.1, U4.6 (CLK2)
