File: CW HF Transceiver.kicad_pcb (KiCad board)
At the start: 2 copper layers, 0 parts

Commit message: some big updates
Parts:
- added C1: 22u, Capacitor_SMD:C_0603_1608Metric, F.Cu at (127.8, 97.9)
- added C10: 1u, Capacitor_SMD:C_0603_1608Metric, F.Cu at (131.8, 105.4)
- added C11: 100n, Capacitor_SMD:C_0603_1608Metric, F.Cu at (131.8, 107.9)
- added C12: 100n, Capacitor_SMD:C_0603_1608Metric, F.Cu at (131.8, 110.4)
- added C13: 100n, Capacitor_SMD:C_0603_1608Metric, F.Cu at (135.8, 97.9)
- added C14: 100n, Capacitor_SMD:C_0603_1608Metric, F.Cu at (135.8, 100.4)
- added C15: 100n, Capacitor_SMD:C_0603_1608Metric, F.Cu at (135.8, 102.9)
- added C16: 100n, Capacitor_SMD:C_0603_1608Metric, F.Cu at (135.8, 105.4)
- added C17: 1p, Capacitor_SMD:C_0603_1608Metric, F.Cu at (177.1, 65.0)
- added C18: 1p, Capacitor_SMD:C_0603_1608Metric, F.Cu at (177.1, 67.5)
- added C19: 1u, Capacitor_SMD:C_0603_1608Metric, F.Cu at (165.7, 102.5)
- added C2: 22u, Capacitor_SMD:C_0603_1608Metric, F.Cu at (127.8, 100.4)
- added C20: 1u, Capacitor_SMD:C_0603_1608Metric, F.Cu at (165.7, 105.0)
- added C21: 22u, Capacitor_SMD:C_0603_1608Metric, F.Cu at (173.6, 46.4)
- added C22: 22u, Capacitor_SMD:C_0603_1608Metric, F.Cu at (173.6, 48.9)
- added C23: 100n, Capacitor_SMD:C_0603_1608Metric, F.Cu at (173.6, 51.4)
- added C24: 22p, Capacitor_SMD:C_0603_1608Metric, F.Cu at (117.8, 97.9)
- added C25: 22p, Capacitor_SMD:C_0603_1608Metric, F.Cu at (117.8, 100.4)
- added C26: 22n, Capacitor_SMD:C_0603_1608Metric, F.Cu at (117.8, 102.9)
- added C27: 100n, Capacitor_SMD:C_0603_1608Metric, F.Cu at (117.8, 105.4)
- added C28: 100n, Capacitor_SMD:C_0603_1608Metric, F.Cu at (117.8, 107.9)
- added C3: 100n, Capacitor_SMD:C_0603_1608Metric, F.Cu at (127.8, 102.9)
- added C4: 15p, Capacitor_SMD:C_0603_1608Metric, F.Cu at (127.8, 105.4)
- added C5: 15p, Capacitor_SMD:C_0603_1608Metric, F.Cu at (127.8, 107.9)
- added C6: 100n, Capacitor_SMD:C_0603_1608Metric, F.Cu at (127.8, 110.4)
- added C7: 100n, Capacitor_SMD:C_0603_1608Metric, F.Cu at (131.8, 97.9)
- added C8: 1u, Capacitor_SMD:C_0603_1608Metric, F.Cu at (131.8, 100.4)
- added C9: 100n, Capacitor_SMD:C_0603_1608Metric, F.Cu at (131.8, 102.9)
- added D1: D_Zener, Diode_SMD:D_0805_2012Metric, F.Cu at (158.1, 59.2)
- added D2: D, Diode_SMD:D_0805_2012Metric, F.Cu at (140.0, 119.9)
- added J1: Barrel_Jack, Connector_BarrelJack:BarrelJack_SwitchcraftConxall_RAPC10U_Horizontal, F.Cu at (161.1, 48.1)
- added J3: AudioJack2, Connector_Audio:Jack_speakON-6.35mm_Neutrik_NLJ2MDXX-H_Horizontal, F.Cu at (94.1, 49.4)
- added J4: AudioJack3, Connector_Audio:Jack_XLR_Neutrik_NC3FAAH-0_Horizontal, F.Cu at (139.4, 67.4)
- added J5: Conn_Coaxial, Connector_Audio:Jack_speakON-6.35mm_Neutrik_NLJ2MDXX-H_Horizontal, F.Cu at (51.5, 78.8)
- added J7: AudioJack3, Connector_Audio:Jack_XLR_Neutrik_NC3FAAH-0_Horizontal, F.Cu at (99.6, 106.5)
- added JP1: Reset, Jumper:SolderJumper-2_P1.3mm_Open_RoundedPad1.0x1.5mm, F.Cu at (146.1, 118.5)
- added L1: 396u, Inductor_SMD:L_0603_1608Metric, F.Cu at (177.1, 70.0)
- added L2: 28.1u, Inductor_SMD:L_0603_1608Metric, F.Cu at (177.1, 72.5)
- added LS1: Speaker, Inductor_SMD:L_0603_1608Metric, F.Cu at (117.8, 110.4)
- added Q1: DMN13H750S, Package_TO_SOT_SMD:SOT-23, F.Cu at (167.6, 66.1)
- added Q2: DMN13H750S, Package_TO_SOT_SMD:SOT-23, F.Cu at (167.6, 70.7)
- added Q3: DMN13H750S, Package_TO_SOT_SMD:SOT-23, F.Cu at (167.6, 75.3)
- added Q4: DMN13H750S, Package_TO_SOT_SMD:SOT-23, F.Cu at (167.6, 80.0)
- added Q5: BS170, Package_TO_SOT_THT:TO-92_Inline, F.Cu at (167.1, 41.8)
- added Q6: BS170, Package_TO_SOT_THT:TO-92_Inline, F.Cu at (167.1, 47.6)
- added Q7: BS170, Package_TO_SOT_THT:TO-92_Inline, F.Cu at (167.1, 53.4)
- added Q8: BS170, Package_TO_SOT_THT:TO-92_Inline, F.Cu at (167.1, 59.2)
- added R1: R, Resistor_SMD:R_0805_2012Metric, F.Cu at (158.1, 62.2)
- added R10: 1k, Resistor_SMD:R_0805_2012Metric, F.Cu at (148.8, 104.0)
- added R11: 4.7k, Resistor_SMD:R_0603_1608Metric, F.Cu at (117.8, 113.0)
- added R12: 4.7k, Resistor_SMD:R_0603_1608Metric, F.Cu at (157.9, 64.9)
- added R2: 5k1, Resistor_SMD:R_0805_2012Metric, F.Cu at (140.0, 98.1)
- added R3: 5k1, Resistor_SMD:R_0805_2012Metric, F.Cu at (140.0, 101.1)
- added R4: 1k, Resistor_SMD:R_0805_2012Metric, F.Cu at (140.0, 104.0)
- added R5: 10k, Resistor_SMD:R_0805_2012Metric, F.Cu at (144.4, 98.1)
- added R6: 27.4, Resistor_SMD:R_0805_2012Metric, F.Cu at (144.4, 101.1)
- added R7: 27.4, Resistor_SMD:R_0805_2012Metric, F.Cu at (144.4, 104.0)
- added R8: 1k, Resistor_SMD:R_0805_2012Metric, F.Cu at (148.8, 98.1)
- added R9: 1k, Resistor_SMD:R_0805_2012Metric, F.Cu at (148.8, 101.1)
- added SW2: Reset RX, Button_Switch_SMD:SW_Push_1P1T_NO_6x6mm_H9.5mm, F.Cu at (97.1, 127.5)
- added TP1: Filters In, TestPoint:TestPoint_Pad_D3.0mm, F.Cu at (172.5, 66.2)
- added TP2: Filters out, TestPoint:TestPoint_Pad_D3.0mm, F.Cu at (172.5, 71.3)
- added TP3: CLK0, TestPoint:TestPoint_Pad_D3.0mm, F.Cu at (161.2, 99.2)
- added TP4: CLK2, TestPoint:TestPoint_Pad_D3.0mm, F.Cu at (161.2, 104.2)
- added TP5: CLK1, TestPoint:TestPoint_Pad_D3.0mm, F.Cu at (161.2, 109.3)
- added TP6: Amp Out, TestPoint:TestPoint_Pad_D3.0mm, F.Cu at (178.2, 47.6)
- added U1: MCP1700x-330xxMB, Package_TO_SOT_SMD:SOT-89-3, F.Cu at (141.2, 115.4)
- added U2: W25Q128JVS, Package_SO:SOIC-8_5.23x5.23mm_P1.27mm, F.Cu at (143.0, 108.9)
- added U3: RP2040, Package_DFN_QFN:QFN-56-1EP_7x7mm_P0.4mm_EP3.2x3.2mm, F.Cu at (130.4, 116.3)
- added U4: Si5351A-B-GT, Package_SO:MSOP-10_3x3mm_P0.5mm, F.Cu at (167.4, 99.0)
- added U5: MCP1700x-500xxMB, Package_TO_SOT_SMD:SOT-89-3, F.Cu at (175.0, 55.7)
- added U6: 74ACT08, Package_SO:TSSOP-14_4.4x5mm_P0.65mm, F.Cu at (176.0, 41.8)
- added U7: Si4735-D60-GU, Package_SO:SSOP-24_3.9x8.7mm_P0.635mm, F.Cu at (119.8, 119.4)
- added Y1: ABM8-272-T3, Crystal:Crystal_SMD_Abracon_ABM8G-4Pin_3.2x2.5mm, F.Cu at (146.6, 114.5)
- added Y2: 25MHz, Crystal:Crystal_AT310_D3.0mm_L10.0mm_Horizontal, F.Cu at (154.5, 98.0)
- added Y3: 37.628KHz, Crystal:Crystal_SMD_2012-2Pin_2.0x1.2mm, F.Cu at (117.6, 126.0)

Commit message: update
Parts:
- removed D1: D_Zener, Diode_SMD:D_0805_2012Metric
- removed D2: D, Diode_SMD:D_0805_2012Metric
- removed J1: Barrel_Jack, Connector_BarrelJack:BarrelJack_SwitchcraftConxall_RAPC10U_Horizontal
- removed J3: AudioJack2, Connector_Audio:Jack_speakON-6.35mm_Neutrik_NLJ2MDXX-H_Horizontal
- removed J4, J7: AudioJack3, Connector_Audio:Jack_XLR_Neutrik_NC3FAAH-0_Horizontal
- removed J5: Conn_Coaxial, Connector_Audio:Jack_speakON-6.35mm_Neutrik_NLJ2MDXX-H_Horizontal
- removed JP1: Reset, Jumper:SolderJumper-2_P1.3mm_Open_RoundedPad1.0x1.5mm
- removed L1: 396u, Inductor_SMD:L_0603_1608Metric
- removed L2: 28.1u, Inductor_SMD:L_0603_1608Metric
- removed LS1: Speaker, Inductor_SMD:L_0603_1608Metric
- removed Q1, Q2, Q3, Q4: DMN13H750S, Package_TO_SOT_SMD:SOT-23
- removed Q5, Q6, Q7, Q8: BS170, Package_TO_SOT_THT:TO-92_Inline
- removed SW2: Reset RX, Button_Switch_SMD:SW_Push_1P1T_NO_6x6mm_H9.5mm
- removed TP1: Filters In, TestPoint:TestPoint_Pad_D3.0mm
- removed TP2: Filters out, TestPoint:TestPoint_Pad_D3.0mm
- removed TP3: CLK0, TestPoint:TestPoint_Pad_D3.0mm
- removed TP4: CLK2, TestPoint:TestPoint_Pad_D3.0mm
- removed TP5: CLK1, TestPoint:TestPoint_Pad_D3.0mm
- removed TP6: Amp Out, TestPoint:TestPoint_Pad_D3.0mm
- removed U1: MCP1700x-330xxMB, Package_TO_SOT_SMD:SOT-89-3
- removed U2: W25Q128JVS, Package_SO:SOIC-8_5.23x5.23mm_P1.27mm
- removed U3: RP2040, Package_DFN_QFN:QFN-56-1EP_7x7mm_P0.4mm_EP3.2x3.2mm
- removed U6: 74ACT08, Package_SO:TSSOP-14_4.4x5mm_P0.65mm
- removed U7: Si4735-D60-GU, Package_SO:SSOP-24_3.9x8.7mm_P0.635mm
- removed Y1: ABM8-272-T3, Crystal:Crystal_SMD_Abracon_ABM8G-4Pin_3.2x2.5mm
- removed Y2: 25MHz, Crystal:Crystal_AT310_D3.0mm_L10.0mm_Horizontal
- removed Y3: 37.628KHz, Crystal:Crystal_SMD_2012-2Pin_2.0x1.2mm
- R1, R10, R2, R3, R4, R5, R6, R7, R8, R9: footprint Resistor_SMD:R_0805_2012Metric -> Resistor_SMD:R_0603_1608Metric
- moved R11 103.1 mm to (214.7, 77.6)
- moved C24 102.3 mm to (214.7, 65.0)
- moved C25 102.3 mm to (214.7, 67.5)
- moved C26 102.3 mm to (214.7, 70.0)
- moved C27 102.3 mm to (214.7, 72.5)
- moved C28 102.3 mm to (214.7, 75.1)
- moved C15 78.6 mm to (204.7, 65.0)
- moved C16 78.6 mm to (204.7, 67.5)
- moved C10 77.5 mm to (200.7, 70.0)
- moved C11 77.5 mm to (200.7, 72.5)
- moved C12 77.5 mm to (200.7, 75.1)
- moved C8 77.5 mm to (200.7, 65.0)
- moved C9 77.5 mm to (200.7, 67.5)
- moved C1 76.3 mm to (196.7, 65.0)
- moved C2 76.3 mm to (196.7, 67.5)
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Other:
- rule pad_to_mask_clearance: 0 -> 0.038

Commit message: add the pcb
Parts:
- removed R12: 4.7k, Resistor_SMD:R_0603_1608Metric
- added Audio1: PJ-327C-4A, plib:AUDIO-SMD_PJ-327C-4A, F.Cu at (157.8, 53.7)
- added Audio2: PJ-327C-4A, plib:AUDIO-SMD_PJ-327C-4A, F.Cu at (146.6, 53.7)
- added C29: 22n, Capacitor_SMD:C_0603_1608Metric, F.Cu at (123.3, 90.3)
- added C30: 100n, Capacitor_SMD:C_0603_1608Metric, F.Cu at (120.3, 90.3)
- added C31: 100n, Capacitor_SMD:C_0603_1608Metric, F.Cu at (121.8, 88.0)
- added D1: 1N4007, Diode_SMD:D_SOD-123, F.Cu at (133.9, 92.2)
- added D10: 1N4007, Diode_SMD:D_SOD-123F, F.Cu at (151.8, 124.7)
- added D2: 1N4148, Diode_SMD:D_SOD-123, F.Cu at (144.9, 106.3)
- added D3: 1N4148, Diode_SMD:D_SOD-123, F.Cu at (148.3, 103.3)
- added D4: 1N4148, Diode_SMD:D_SOD-123, F.Cu at (148.3, 100.9)
- added D5: 1N4007, Diode_SMD:D_SOD-123F, F.Cu at (120.4, 107.7)
- added D6: 1N4007, Diode_SMD:D_SOD-123F, F.Cu at (117.4, 120.4)
- added D7: 1N4007, Diode_SMD:D_SOD-123F, F.Cu at (139.4, 122.2)
- added D8: 1N4007, Diode_SMD:D_SOD-123F, F.Cu at (134.1, 99.2)
- added D9: 1N4007, Diode_SMD:D_SOD-123F, F.Cu at (135.8, 121.7)
- added H1: MountingHole_Pad, MountingHole:MountingHole_3.2mm_M3_Pad_Via, F.Cu at (119.0, 52.3)
- added H2: MountingHole_Pad, MountingHole:MountingHole_3.2mm_M3_Pad_Via, F.Cu at (119.0, 132.3)
- added H3: MountingHole_Pad, MountingHole:MountingHole_3.2mm_M3_Pad_Via, F.Cu at (179.2, 132.3)
- added H4: MountingHole_Pad, MountingHole:MountingHole_3.2mm_M3_Pad_Via, F.Cu at (179.2, 52.3)
- added J1: JTAG, Connector_PinHeader_1.27mm:PinHeader_1x04_P1.27mm_Vertical, F.Cu at (140.8, 83.2)
- added J2: Conn_02x12_Odd_Even, Connector_PinHeader_1.27mm:PinHeader_2x12_P1.27mm_Vertical_SMD, F.Cu at (120.3, 74.7)
- added J3: Barrel_Jack_Switch, plib:DC-IN-TH_DC-5520-1, F.Cu at (168.6, 55.0)
- added JP1: RST RX, Jumper:SolderJumper-2_P1.3mm_Open_RoundedPad1.0x1.5mm, F.Cu at (118.2, 85.9)
- added L1: L, Inductor_SMD:L_0603_1608Metric, F.Cu at (144.2, 129.5)
- added L10: L, Inductor_SMD:L_0603_1608Metric, F.Cu at (129.6, 109.9)
- added L11: L, Inductor_SMD:L_0603_1608Metric, F.Cu at (146.4, 111.3)
- added L12: 330n, plib:ft37-67, F.Cu at (129.6, 103.5)
- added L13: 560n, plib:ft37-67, F.Cu at (129.5, 117.0)
- added L14: 1.3u, plib:ft37-67, F.Cu at (149.8, 118.2)
- added L15: L, Inductor_SMD:L_0603_1608Metric, F.Cu at (165.4, 128.7)
- added L2: L, Inductor_SMD:L_0603_1608Metric, F.Cu at (141.9, 131.7)
- added L3: L, Inductor_SMD:L_0603_1608Metric, F.Cu at (154.0, 91.0)
- added L4: L, Inductor_SMD:L_0603_1608Metric, F.Cu at (140.2, 90.4)
- added L5: L, Inductor_SMD:L_0603_1608Metric, F.Cu at (158.0, 91.1)
- added L6: 330n, plib:ft37-67, F.Cu at (123.1, 101.0)
- added L7: 560n, plib:ft37-67, F.Cu at (123.0, 114.5)
- added L8: 1.5u, plib:ft37-67, F.Cu at (142.9, 115.9)
- added L9: L, Inductor_SMD:L_0603_1608Metric, F.Cu at (137.5, 100.0)
- added Q1: BSS123, Package_TO_SOT_SMD:SOT-23, F.Cu at (137.6, 104.0)
- added Q10: BSS123, Package_TO_SOT_SMD:SOT-23, F.Cu at (167.9, 85.5)
- added Q11: BSS123, Package_TO_SOT_SMD:SOT-23, F.Cu at (168.0, 70.4)
- added Q12: BSS123, Package_TO_SOT_SMD:SOT-23, F.Cu at (163.9, 85.5)
- added Q13: BSS123, Package_TO_SOT_SMD:SOT-23, F.Cu at (164.0, 70.4)
- added Q2: BSS123, Package_TO_SOT_SMD:SOT-23, F.Cu at (134.3, 113.3)
- added Q3: BSS123, Package_TO_SOT_SMD:SOT-23, F.Cu at (152.0, 110.7)
- added Q4: BSS123, Package_TO_SOT_SMD:SOT-23, F.Cu at (179.9, 85.5)
- added Q5: BSS123, Package_TO_SOT_SMD:SOT-23, F.Cu at (179.9, 70.4)
- added Q6: BSS123, Package_TO_SOT_SMD:SOT-23, F.Cu at (175.9, 85.5)
- added Q7: BSS123, Package_TO_SOT_SMD:SOT-23, F.Cu at (176.0, 70.4)
- added Q8: BSS123, Package_TO_SOT_SMD:SOT-23, F.Cu at (171.9, 85.5)
- added Q9: BSS123, Package_TO_SOT_SMD:SOT-23, F.Cu at (172.1, 70.4)
- added RF1: DOSIN-801-0050, plib:BNC-TH_DOSIN-801-0051, F.Cu at (132.7, 130.7)
- added T1: 1:2, plib:ft50-75 trafo with CT, F.Cu at (168.0, 113.4)
- added TP1: Filters out, TestPoint:TestPoint_Pad_D2.0mm, F.Cu at (137.5, 95.9)
- added TP2: CLK0, TestPoint:TestPoint_Pad_D2.0mm, F.Cu at (158.0, 75.0)
- added TP3: CLK2, TestPoint:TestPoint_Pad_D2.0mm, F.Cu at (158.0, 78.5)
- added TP4: CLK1, TestPoint:TestPoint_Pad_D2.0mm, F.Cu at (158.0, 82.0)
- added TP5: Amp Out, TestPoint:TestPoint_Pad_D2.0mm, F.Cu at (174.9, 93.6)
- added U1: USB6B1, Package_SO:SOIC-8_3.9x4.9mm_P1.27mm, F.Cu at (137.0, 62.4)
- added U2: MCP1700x-330xxMB, Package_TO_SOT_SMD:SOT-89-3, F.Cu at (127.4, 61.9)
- added U3: STM32F072C8Tx, Package_QFP:LQFP-48_7x7mm_P0.5mm, F.Cu at (136.0, 74.0)
- added U6: 74ACT08, Package_DIP:DIP-14_W7.62mm, F.Cu at (164.4, 81.8)
- added U7: Si4735-D60-GU, Package_SO:SSOP-24_3.9x8.7mm_P0.635mm, F.Cu at (128.2, 88.9)
- added USBC1: USB3.1C16PFSMT, plib:USB-C-SMD_TYPE-C-USB-17, F.Cu at (132.8, 52.4)
- added Y1: NX3225GA-25.000M-STD-CRG-2, Crystal:Crystal_SMD_3225-4Pin_3.2x2.5mm, F.Cu at (154.0, 81.7)
- C1, C2: value 22u -> C
- C10: value 1u -> C
- C11, C12, C13, C28: value 100n -> C
- C14: value 100n -> 110p
- C15: value 100n -> 180p
- C16: value 100n -> 470p
- C17: value 1p -> 180p
- C18: value 1p -> 300p
- C19: value 1u -> 750p
- C20: value 1u -> 91p
- C21: value 22u -> 160p
- C22: value 22u -> 430p
- C23: value 100n -> 1u
- C24: value 22p -> 1u
- C25: value 22p -> 22u
- C26: value 22n -> 22u
- C3: value 100n -> 22u
- C4: value 15p -> 22u
- C5: value 15p -> 100n
- C8: value 1u -> 100n
- R1: value R -> 4.7k
- R10, R8, R9: value 1k -> R
- R2: value 5k1 -> 4.7k
- R4: value 1k -> 5k1
- R5: value 10k -> 1k
- R6: value 27.4 -> 1k
- R7: value 27.4 -> R
- moved C18 108.0 mm to (126.2, 119.8), turned to -90 degrees
- moved C17 102.8 mm to (126.5, 106.3), turned to -90 degrees
- moved C15 100.2 mm to (118.8, 116.6), turned to 180 degrees
- moved R11 98.2 mm to (117.2, 89.1), turned to 90 degrees
- moved C20 90.9 mm to (132.5, 106.5), turned to -90 degrees
- moved C14 85.0 mm to (119.1, 104.0), turned to -90 degrees
- moved C19 83.5 mm to (146.9, 121.0), turned to -90 degrees
- moved C16 82.8 mm to (139.6, 118.7), turned to -90 degrees
- moved R9 82.8 mm to (137.4, 112.1), turned to 90 degrees
- moved C2 80.2 mm to (146.6, 130.2), turned to -90 degrees
- moved R3 76.5 mm to (129.7, 57.4), turned to 180 degrees
- moved R8 75.3 mm to (141.3, 101.1), turned to 90 degrees
- moved C28 75.1 mm to (162.1, 128.7), turned to 180 degrees
- moved R1 73.1 mm to (143.8, 64.4), turned to 180 degrees
- moved C21 72.4 mm to (133.5, 120.0), turned to -90 degrees
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Connections:
- C1 pad 1: +5V -> /Receiver/Input
- C1 pad 2: GND -> /Filtering/t/r rbias
- C10 pad 1: +3.3V -> VCC
- C11 pad 1: +3.3V -> /Filtering/Input Bias
- C11 pad 2: Net-(C11-Pad2) -> Net-(D2-K)
- C12 pad 1: +3.3V -> GND
- C12 pad 2: Net-(C11-Pad2) -> /Filtering/voltage tripler
- C13 pad 1: +3.3V -> VCC
- C13 pad 2: Net-(C11-Pad2) -> GND
- C14 pad 1: +3.3V -> Net-(D5-K)
- C14 pad 2: Net-(C11-Pad2) -> GND
- C15 pad 1: +3.3V -> Net-(D6-K)
- C15 pad 2: Net-(C11-Pad2) -> GND
- C16 pad 1: +3.3V -> Net-(D7-K)
- C16 pad 2: Net-(C11-Pad2) -> GND
- C19 pad 1: +3.3V -> Net-(C19-Pad1)
- C2 pad 1: +3.3V -> /Filtering/Output Bias
- C2 pad 2: GND -> /ant
- C20 pad 1: VCC -> Net-(D8-K)
- C21 pad 1: Vdrive -> Net-(D9-K)
- C22 pad 1: +5V -> Net-(D10-K)
- C23 pad 1: +5V -> +3.3V
- C24 pad 1: /Receiver/DCLK -> +3.3V
- C25 pad 1: /Receiver/RCLK -> VCC
- C26 pad 1: +3.3V -> +5V
- C26 pad 2: Net-(U7-DBYP) -> GND
- C27 pad 1: +3.3V -> +5V
- C28 pad 1: +3.3V -> VCC
- C3 pad 1: +3.3V -> +5V
- C4 pad 1: GND -> +3.3V
- C4 pad 2: Net-(U3-XIN) -> GND
- C5 pad 1: GND -> +3.3V
- C5 pad 2: Net-(C5-Pad2) -> GND
- C6 pad 1: +1V1 -> +3.3V
- C7 pad 1: +1V1 -> +3.3V
- C8 pad 1: +1V1 -> +3.3V
- C9 pad 2: Net-(C11-Pad2) -> GND
- R1 pad 1: VCC -> +3.3V
- R1 pad 2: Vdrive -> /dit
- R10 pad 1: +3.3V -> Net-(Q3-D)
- R10 pad 2: /RP2040 Driver/sda -> /Filtering/voltage tripler
- R2 pad 1: Net-(J6-CC2) -> +3.3V
- R2 pad 2: GND -> /dah
- R4 pad 2: /RP2040 Driver/QSPI_SS -> GND
- R5 pad 2: /RP2040 Driver/QSPI_SS -> /STM32 Driver/scl
- R6 pad 1: /RP2040 Driver/D+ -> +3.3V
- R6 pad 2: Net-(U3-USB_DP) -> /STM32 Driver/sda
- R7 pad 1: /RP2040 Driver/D- -> /Filtering/voltage tripler
- R8 pad 1: Net-(C5-Pad2) -> Net-(Q1-D)
- R8 pad 2: Net-(U3-XOUT) -> /Filtering/voltage tripler
- R9 pad 1: +3.3V -> Net-(Q2-D)
- R9 pad 2: /RP2040 Driver/scl -> /Filtering/voltage tripler
- U4 pad 4: /RP2040 Driver/scl -> /STM32 Driver/scl
- U4 pad 5: /RP2040 Driver/sda -> /STM32 Driver/sda
- U4 pad 6: /Square Wave Gen/BFO out -> /Receiver/Receiver clk
- U5 pad 2: Vdrive -> VCC
Routing:
- net VCC: track 0.00 -> 169.4 mm, vias 0 -> 14
- net +3.3V: track 0.00 -> 141.6 mm, vias 0 -> 11
- net /Filtering/Input Bias: track 0.00 -> 106.0 mm, vias 0 -> 3
- net /Filtering/Output Bias: track 0.00 -> 86.8 mm, vias 0 -> 2
- net /Receiver/Rout: track 0.00 -> 82.2 mm
- net /Receiver/Lout: track 0.00 -> 71.4 mm
- net +5V: track 0.00 -> 63.2 mm, vias 0 -> 3
- net /STM32 Driver/scl: track 0.00 -> 62.3 mm, vias 0 -> 5
- net /STM32 Driver/sda: track 0.00 -> 61.6 mm, vias 0 -> 4
- net /Amplifier/Amp enable: track 0.00 -> 58.8 mm, vias 0 -> 3
- net GND: track 0.00 -> 58.7 mm, vias 0 -> 166
- net /Receiver/Receiver clk: track 0.00 -> 50.0 mm, vias 0 -> 2
- net /Amplifier/180º Wave: track 0.00 -> 48.9 mm
- net /Filtering/Filter 3 En: track 0.00 -> 43.6 mm, vias 0 -> 2
- net /Filtering/Filter 2 En: track 0.00 -> 43.2 mm, vias 0 -> 2
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- added copper zone on B.Cu, net GND
- added copper zone on F.Cu, net GND
Other:
- board outline added: 70.2 x 90 mm
- board text added: "S"

Commit message: a
Routing:
- net GND: vias 166 -> 358
