File: Schematics/CW HF Transceiver.kicad_sch (KiCad schematic)
At the start: 7 parts, among them J1 Barrel_Jack, J2 AudioJack3, J3 Conn_Coaxial

Commit message: Reformating
Parts:
- removed D1: D_Zener, symbol Device:D_Zener
Connections:
- no-connect marks 1 -> 0
