File: Schematics/IO.kicad_sch (KiCad schematic)
At the start: 2 parts, among them SW1 VFO

Commit message: Reformating
Parts:
- RV1: value AF Gain -> Volume
Changed lines of the file:
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@@
 	(symbol
 		(lib_id "Device:R_Potentiometer")
-		(at 107.95 106.68 0)
+		(at 113.03 105.41 0)
 		(unit 1)
 		(exclude_from_sim no)
@@
 		(fields_autoplaced yes)
 		(property "Reference" "RV1"
-			(at 105.41 105.4099 0)
+			(at 110.49 104.1399 0)
 			(effects
 				(font
@@
 			)
 		)
-		(property "Value" "AF Gain"
-			(at 105.41 107.9499 0)
+		(property "Value" "Volume"
+			(at 110.49 106.6799 0)
 			(effects
 				(font
@@
 		)
 		(property "Footprint" ""
-			(at 107.95 106.68 0)
+			(at 113.03 105.41 0)
 			(effects
 				(font
@@
 		)
 		(property "Datasheet" "~"
-			(at 107.95 106.68 0)
+			(at 113.03 105.41 0)
 			(effects
 				(font
@@
 		)
 		(property "Description" "Potentiometer"
-			(at 107.95 106.68 0)
+			(at 113.03 105.41 0)
 			(effects
 				(font
