File: Schematics/STM32 Driver.kicad_sch (KiCad schematic)
At the start: 16 parts, among them J4 USB_C_Receptacle_USB2.0_14P, U1 MCP1700x-330xxMB, U2 STM32F072C8Tx

Commit message: Reformating
Parts:
- added TP8: SWCLK, symbol Connector:TestPoint
- added U7: USB6B1, Package_SO:SOIC-8_3.9x4.9mm_P1.27mm, symbol Power_Protection:USB6B1
Connections:
- net D+: now also U2.32 (PA11), U7.6 (I/O2); no longer U2.33 (PA12)
- net D-: now also U2.33 (PA12), U7.7 (I/O1); no longer U2.32 (PA11)
- net GND: now also U7.4 (GND), U7.5 (GND)
- net at U2.37 (PA14): now also TP8.1
- net VBUS: now reaches D2.2 (A), J4.A4 (VBUS), J4.A9 (VBUS), J4.B4 (VBUS), J4.B9 (VBUS)
- net VBUS: now also U7.1 (VBUS), U7.8 (VBUS)
- net at J4.A6 (D+), J4.B6 (D+): now also U7.3 (I/O2)
- net at J4.A7 (D-), J4.B7 (D-): now also U7.2 (I/O1)
- no-connect marks 29 -> 28
Other:
- moved on the sheet: D2
